File: TSC BW 16 V3.1/Ethernet_W5500.kicad_sch (KiCad schematic)
At the start: 36 parts, among them J16 RJ45_Hanrun_HR911105A_Horizon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, U45 W5500, Y3 25M

Commit message: WORKING ON IT
Other:
- note added: "ETHERNET GLOBAL PINS / LABELS P15"
- note added: "Ethernet (W5500) ETH_SCLK - PIN35 : GPIO42 ETH_MOSI - PIN37 : GPIO43 ETH_MISO - PIN36 : GPIO44 ETH_SCS - PIN8 : GPIO15 ETH_INT - PIN38 : GPIO2 ETH_RST - PIN39 : GPIO1"
- note removed: "GLOBAL PINS / LABELS"
- note removed: "ethernet: type: W5500 clk_pin: GPIO42 mosi_pin: GPIO43 miso_pin: GPIO44 cs_pin: GPIO15 interrupt_pin: GPIO2 reset_pin: GPIO1"
Changed lines of the file:
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@@
 	)
 	(rectangle
-		(start 129.54 149.86)
-		(end 165.1 186.69)
+		(start 17.78 148.59)
+		(end 54.61 193.04)
 		(stroke
 			(width 1)
@@
 		)
 	)
-	(text "ethernet:\n  type: W5500\n  clk_pin: GPIO42\n  mosi_pin: GPIO43\n  miso_pin: GPIO44\n  cs_pin: GPIO15\n  interrupt_pin: GPIO2\n  reset_pin: GPIO1\n"
+	(text "ETHERNET GLOBAL PINS / LABELS P15"
 		(exclude_from_sim no)
-		(at 112.268 172.72 0)
-		(effects
-			(font
-				(size 1.27 1.27)
-			)
-		)
-	)
-	(text "GLOBAL PINS / LABELS"
+		(at 35.306 145.542 0)
+		(effects
+			(font
+				(size 1.27 1.27)
+			)
+		)
+	)
+	(text "Ethernet (W5500)\nETH_SCLK - PIN35 : GPIO42\nETH_MOSI - PIN37 : GPIO43\nETH_MISO - PIN36 : GPIO44\nETH_SCS - PIN8 : GPIO15\nETH_INT - PIN38 : GPIO2\nETH_RST - PIN39 : GPIO1"
 		(exclude_from_sim no)
-		(at 147.32 155.448 0)
-		(effects
-			(font
-				(size 1.27 1.27)
-			)
+		(at 22.352 182.88 0)
+		(effects
+			(font
+				(size 1.27 1.27)
+				(color 33 191 7 1)
+			)
+			(justify left)
 		)
 	)
@@
 	(wire
 		(pts
-			(xy 135.89 179.07) (xy 149.86 179.07)
-		)
-		(stroke
-			(width 0)
-			(type default)
-		)
-	)
-	(wire
-		(pts
 			(xy 39.37 110.49) (xy 35.56 110.49)
 		)
@@
 	(wire
 		(pts
-			(xy 135.89 175.26) (xy 149.86 175.26)
-		)
-		(stroke
-			(width 0)
-			(type default)
-		)
-	)
-	(wire
-		(pts
 			(xy 156.21 86.36) (xy 156.21 88.9)
 		)
@@
 	(wire
 		(pts
+			(xy 21.59 152.4) (xy 35.56 152.4)
+		)
+		(stroke
+			(width 0)
+			(type default)
+		)
+	)
+	(wire
+		(pts
 			(xy 265.43 88.9) (xy 270.51 88.9)
 		)
@@
 	(wire
 		(pts
+			(xy 21.59 171.45) (xy 35.56 171.45)
+		)
+		(stroke
+			(width 0)
+			(type default)
+		)
+	)
+	(wire
+		(pts
 			(xy 227.33 74.93) (xy 256.54 74.93)
 		)
@@
 	(wire
 		(pts
-			(xy 135.89 160.02) (xy 149.86 160.02)
-		)
-		(stroke
-			(width 0)
-			(type default)
-		)
-	)
-	(wire
-		(pts
 			(xy 62.23 93.98) (xy 74.93 93.98)
 		)
@@
 	(wire
 		(pts
-			(xy 135.89 167.64) (xy 149.86 167.64)
-		)
-		(stroke
-			(width 0)
-			(type default)
-		)
-	)
-	(wire
-		(pts
 			(xy 116.84 134.62) (xy 119.38 134.62)
 		)
@@
 	(wire
 		(pts
+			(xy 21.59 167.64) (xy 35.56 167.64)
+		)
+		(stroke
+			(width 0)
+			(type default)
+		)
+	)
+	(wire
+		(pts
 			(xy 76.2 38.1) (xy 88.9 38.1)
 		)
@@
 	(wire
 		(pts
-			(xy 135.89 171.45) (xy 149.86 171.45)
-		)
-		(stroke
-			(width 0)
-			(type default)
-		)
-	)
-	(wire
-		(pts
 			(xy 227.33 63.5) (xy 256.54 63.5)
 		)
@@
 	(wire
 		(pts
+			(xy 21.59 156.21) (xy 35.56 156.21)
+		)
+		(stroke
+			(width 0)
+			(type default)
+		)
+	)
+	(wire
+		(pts
 			(xy 31.75 82.55) (xy 29.21 82.55)
 		)
@@
 	(wire
 		(pts
+			(xy 21.59 163.83) (xy 35.56 163.83)
+		)
+		(stroke
+			(width 0)
+			(type default)
+		)
+	)
+	(wire
+		(pts
 			(xy 100.33 38.1) (xy 100.33 36.83)
 		)
@@
 	(wire
 		(pts
-			(xy 135.89 163.83) (xy 149.86 163.83)
-		)
-		(stroke
-			(width 0)
-			(type default)
-		)
-	)
-	(wire
-		(pts
 			(xy 180.34 91.44) (xy 194.31 91.44)
 		)
@@
 		(pts
 			(xy 52.07 21.59) (xy 52.07 27.94)
+		)
+		(stroke
+			(width 0)
+			(type default)
+		)
+	)
+	(wire
+		(pts
+			(xy 21.59 160.02) (xy 35.56 160.02)
 		)
 		(stroke
@@
 		)
 	)
+	(label "ETH_INT"
+		(at 24.13 167.64 0)
+		(effects
+			(font
+				(size 1.27 1.27)
+			)
+			(justify left bottom)
+		)
+	)
 	(label "RXN-"
 		(at 205.74 74.93 0)
@@
 		)
 	)
-	(label "ETH_MOSI"
-		(at 138.43 171.45 0)
-		(effects
-			(font
-				(size 1.27 1.27)
-			)
-			(justify left bottom)
-		)
-	)
 	(label "ETH_INT"
 		(at 64.77 96.52 0)
@@
 		)
 	)
-	(label "ETH_SCLK"
-		(at 138.43 163.83 0)
-		(effects
-			(font
-				(size 1.27 1.27)
-			)
-			(justify left bottom)
-		)
-	)
-	(label "ETH_INT"
-		(at 138.43 175.26 0)
-		(effects
-			(font
-				(size 1.27 1.27)
-			)
-			(justify left bottom)
-		)
-	)
 	(label "RD+"
 		(at 246.38 53.34 0)
@@
 		)
 	)
+	(label "ETH_SCLK"
+		(at 24.13 156.21 0)
+		(effects
+			(font
+				(size 1.27 1.27)
+			)
+			(justify left bottom)
+		)
+	)
 	(label "X0"
 		(at 43.18 125.73 0)
@@
 		)
 	)
+	(label "ETH_MOSI"
+		(at 24.13 163.83 0)
+		(effects
+			(font
+				(size 1.27 1.27)
+			)
+			(justify left bottom)
+		)
+	)
 	(label "RD+"
 		(at 185.42 93.98 0)
@@
 		)
 	)
-	(label "ETH_MISO"
-		(at 138.43 167.64 0)
-		(effects
-			(font
-				(size 1.27 1.27)
-			)
-			(justify left bottom)
-		)
-	)
 	(label "TD-"
 		(at 185.42 91.44 0)
@@
 		)
 	)
+	(label "ETH_SCS"
+		(at 24.13 152.4 0)
+		(effects
+			(font
+				(size 1.27 1.27)
+			)
+			(justify left bottom)
+		)
+	)
 	(label "RD-"
 		(at 185.42 99.06 0)
@@
 		)
 	)
-	(label "ETH_SCS"
-		(at 138.43 160.02 0)
-		(effects
-			(font
-				(size 1.27 1.27)
-			)
-			(justify left bottom)
-		)
-	)
 	(label "ActLed"
 		(at 107.95 124.46 0)
@@
 		)
 	)
-	(label "ETH_RST"
-		(at 138.43 179.07 0)
-		(effects
-			(font
-				(size 1.27 1.27)
-			)
-			(justify left bottom)
-		)
-	)
 	(label "X1"
 		(at 68.58 114.3 0)
@@
 		)
 	)
+	(label "ETH_MISO"
+		(at 24.13 160.02 0)
+		(effects
+			(font
+				(size 1.27 1.27)
+			)
+			(justify left bottom)
+		)
+	)
 	(label "RCT"
 		(at 185.42 96.52 0)
@@
 		)
 	)
-	(global_label "ETH_SCLK"
+	(label "ETH_RST"
+		(at 24.13 171.45 0)
+		(effects
+			(font
+				(size 1.27 1.27)
+			)
+			(justify left bottom)
+		)
+	)
+	(global_label "ETH_INT"
 		(shape input)
-		(at 149.86 163.83 0)
+		(at 35.56 167.64 0)
 		(fields_autoplaced yes)
 		(effects
@@
 		)
 		(property "Intersheetrefs" "${INTERSHEET_REFS}"
-			(at 162.0375 163.83 0)
+			(at 45.8628 167.64 0)
 			(hide yes)
 			(show_name no)
@@
 		)
 	)
-	(global_label "ETH_RST"
+	(global_label "ETH_SCS"
 		(shape input)
-		(at 149.86 179.07 0)
+		(at 35.56 152.4 0)
 		(fields_autoplaced yes)
 		(effects
@@
 		)
 		(property "Intersheetrefs" "${INTERSHEET_REFS}"
-			(at 160.707 179.07 0)
+			(at 46.6489 152.4 0)
 			(hide yes)
 			(show_name no)
@@
 		)
 	)
-	(global_label "ETH_INT"
+	(global_label "ETH_MISO"
 		(shape input)
-		(at 149.86 175.26 0)
+		(at 35.56 160.02 0)
 		(fields_autoplaced yes)
 		(effects
@@
 		)
 		(property "Intersheetrefs" "${INTERSHEET_REFS}"
-			(at 160.1628 175.26 0)
+			(at 47.5561 160.02 0)
 			(hide yes)
 			(show_name no)
@@
 		)
 	)
-	(global_label "ETH_SCS"
+	(global_label "ETH_SCLK"
 		(shape input)
-		(at 149.86 160.02 0)
+		(at 35.56 156.21 0)
 		(fields_autoplaced yes)
 		(effects
@@
 		)
 		(property "Intersheetrefs" "${INTERSHEET_REFS}"
-			(at 160.9489 160.02 0)
+			(at 47.7375 156.21 0)
 			(hide yes)
 			(show_name no)
@@
 		)
 	)
-	(global_label "ETH_MISO"
+	(global_label "ETH_RST"
 		(shape input)
-		(at 149.86 167.64 0)
+		(at 35.56 171.45 0)
 		(fields_autoplaced yes)
 		(effects
@@
 		)
 		(property "Intersheetrefs" "${INTERSHEET_REFS}"
-			(at 161.8561 167.64 0)
+			(at 46.407 171.45 0)
 			(hide yes)
 			(show_name no)
@@
 	(global_label "ETH_MOSI"
 		(shape input)
-		(at 149.86 171.45 0)
+		(at 35.56 163.83 0)
 		(fields_autoplaced yes)
 		(effects
@@
 		)
 		(property "Intersheetrefs" "${INTERSHEET_REFS}"
-			(at 161.8561 171.45 0)
+			(at 47.5561 163.83 0)
 			(hide yes)
 			(show_name no)
