File: TSC BW 16 V3.1/RS485 v2.kicad_sch (KiCad schematic)
At the start: 20 parts, among them J15 691312510002, J17 691312510002, U47 MAX13487EESA, U48 MAX13487EESA

Commit message: WORKING ON IT
Other:
- note added: "RS485 TXD - PIN9 : GPIO16 RXD - PIN10 : GPIO17 TXD - PIN23 : GPIO21"
Changed lines of the file:
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@@
 	)
 	(rectangle
-		(start 222.25 96.52)
-		(end 255.27 119.38)
+		(start 228.6 96.52)
+		(end 261.62 135.89)
 		(stroke
 			(width 1)
@@
 	(text "GLOBAL PINS / LABELS"
 		(exclude_from_sim no)
-		(at 239.014 100.33 0)
+		(at 245.364 100.33 0)
 		(effects
 			(font
@@
 		)
 	)
+	(text "RS485\nTXD - PIN9 : GPIO16\nRXD - PIN10 : GPIO17\nTXD - PIN23 : GPIO21"
+		(exclude_from_sim no)
+		(at 233.172 125.73 0)
+		(effects
+			(font
+				(size 1.27 1.27)
+				(color 33 191 7 1)
+			)
+			(justify left)
+		)
+	)
 	(junction
 		(at 213.36 135.89)
@@
 	(wire
 		(pts
-			(xy 227.33 114.3) (xy 240.03 114.3)
+			(xy 233.68 114.3) (xy 246.38 114.3)
 		)
 		(stroke
@@
 	(wire
 		(pts
-			(xy 227.33 104.14) (xy 240.03 104.14)
+			(xy 233.68 104.14) (xy 246.38 104.14)
 		)
 		(stroke
@@
 	(wire
 		(pts
-			(xy 227.33 109.22) (xy 240.03 109.22)
+			(xy 233.68 109.22) (xy 246.38 109.22)
 		)
 		(stroke
@@
 	)
 	(label "485_EN"
-		(at 229.87 109.22 0)
+		(at 236.22 109.22 0)
 		(effects
 			(font
@@
 	)
 	(label "485RX"
-		(at 229.87 114.3 0)
+		(at 236.22 114.3 0)
 		(effects
 			(font
@@
 	)
 	(label "485TX"
-		(at 229.87 104.14 0)
+		(at 236.22 104.14 0)
 		(effects
 			(font
@@
 	(global_label "485_EN"
 		(shape input)
-		(at 240.03 109.22 0)
+		(at 246.38 109.22 0)
 		(fields_autoplaced yes)
 		(effects
@@
 		)
 		(property "Intersheetrefs" "${INTERSHEET_REFS}"
-			(at 250.0908 109.22 0)
+			(at 256.4408 109.22 0)
 			(hide yes)
 			(show_name no)
@@
 	(global_label "485TX"
 		(shape input)
-		(at 240.03 104.14 0)
+		(at 246.38 104.14 0)
 		(fields_autoplaced yes)
 		(effects
@@
 		)
 		(property "Intersheetrefs" "${INTERSHEET_REFS}"
-			(at 248.8208 104.14 0)
+			(at 255.1708 104.14 0)
 			(hide yes)
 			(show_name no)
@@
 	(global_label "485RX"
 		(shape input)
-		(at 240.03 114.3 0)
+		(at 246.38 114.3 0)
 		(fields_autoplaced yes)
 		(effects
@@
 		)
 		(property "Intersheetrefs" "${INTERSHEET_REFS}"
-			(at 249.1232 114.3 0)
+			(at 255.4732 114.3 0)
 			(hide yes)
 			(show_name no)
