File: TSC BW 16 V3.1/RS485.kicad_sch (KiCad schematic)
At the start: 9 parts, among them J12 691312510002, U43 SN65HVD75

Commit message: WORKING ON IT
Other:
- note added: "GLOBAL PINS / LABELS"
- note added: "RS485 TXD - PIN9 : GPIO16 RXD - PIN10 : GPIO17 TXD - PIN23 : GPIO21"
Changed lines of the file:
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@@
 		(comment 4 "Designed by: Lucas Tivana")
+	)
+	(rectangle
+		(start 231.14 119.38)
+		(end 264.16 158.75)
+		(stroke
+			(width 1)
+			(type solid)
+			(color 225 0 0 1)
+		)
+		(fill
+			(type none)
+		)
 	)
 	(text "#define RS485_EN 21\n\nvoid rs485Transmit()\n{\n    digitalWrite(RS485_EN, HIGH);\n}\n\nvoid rs485Receive()\n{\n    digitalWrite(RS485_EN, LOW);\n}\n\nvoid sendRS485(String msg)\n{\n    rs485Transmit();\n    Serial2.print(msg);\n    Serial2.flush();\n    rs485Receive();\n}"
@@
 				(size 1.27 1.27)
 			)
+		)
+	)
+	(text "GLOBAL PINS / LABELS"
+		(exclude_from_sim no)
+		(at 247.904 123.19 0)
+		(effects
+			(font
+				(size 1.27 1.27)
+			)
+		)
+	)
+	(text "RS485\nTXD - PIN9 : GPIO16\nRXD - PIN10 : GPIO17\nTXD - PIN23 : GPIO21"
+		(exclude_from_sim no)
+		(at 235.712 148.59 0)
+		(effects
+			(font
+				(size 1.27 1.27)
+				(color 33 191 7 1)
+			)
+			(justify left)
 		)
 	)
@@
 	(wire
 		(pts
+			(xy 236.22 132.08) (xy 248.92 132.08)
+		)
+		(stroke
+			(width 0)
+			(type default)
+		)
+	)
+	(wire
+		(pts
 			(xy 173.99 115.57) (xy 194.31 115.57)
 		)
@@
 	(wire
 		(pts
+			(xy 236.22 127) (xy 248.92 127)
+		)
+		(stroke
+			(width 0)
+			(type default)
+		)
+	)
+	(wire
+		(pts
 			(xy 140.97 82.55) (xy 140.97 87.63)
 		)
@@
 		(pts
 			(xy 173.99 105.41) (xy 173.99 115.57)
+		)
+		(stroke
+			(width 0)
+			(type default)
+		)
+	)
+	(wire
+		(pts
+			(xy 236.22 137.16) (xy 248.92 137.16)
 		)
 		(stroke
@@
 		)
 	)
+	(label "485_EN"
+		(at 238.76 132.08 0)
+		(effects
+			(font
+				(size 1.27 1.27)
+			)
+			(justify left bottom)
+		)
+	)
 	(label "RS485+"
 		(at 185.42 115.57 0)
@@
 			)
 			(justify left bottom)
+		)
+	)
+	(label "485RX"
+		(at 238.76 137.16 0)
+		(effects
+			(font
+				(size 1.27 1.27)
+			)
+			(justify left bottom)
+		)
+	)
+	(label "485TX"
+		(at 238.76 127 0)
+		(effects
+			(font
+				(size 1.27 1.27)
+			)
+			(justify left bottom)
+		)
+	)
+	(global_label "485_EN"
+		(shape input)
+		(at 248.92 132.08 0)
+		(fields_autoplaced yes)
+		(effects
+			(font
+				(size 1.27 1.27)
+			)
+			(justify left)
+		)
+		(property "Intersheetrefs" "${INTERSHEET_REFS}"
+			(at 258.9808 132.08 0)
+			(hide yes)
+			(show_name no)
+			(do_not_autoplace no)
+			(effects
+				(font
+					(size 1.27 1.27)
+				)
+				(justify left)
+			)
 		)
 	)
@@
 		)
 	)
+	(global_label "485TX"
+		(shape input)
+		(at 248.92 127 0)
+		(fields_autoplaced yes)
+		(effects
+			(font
+				(size 1.27 1.27)
+			)
+			(justify left)
+		)
+		(property "Intersheetrefs" "${INTERSHEET_REFS}"
+			(at 257.7108 127 0)
+			(hide yes)
+			(show_name no)
+			(do_not_autoplace no)
+			(effects
+				(font
+					(size 1.27 1.27)
+				)
+				(justify left)
+			)
+		)
+	)
 	(global_label "MCU_Tx_RS485"
 		(shape input)
@@
 			)
 		)
+	)
+	(global_label "485RX"
+		(shape input)
+		(at 248.92 137.16 0)
+		(fields_autoplaced yes)
+		(effects
+			(font
+				(size 1.27 1.27)
+			)
+			(justify left)
+		)
+		(property "Intersheetrefs" "${INTERSHEET_REFS}"
+			(at 258.0132 137.16 0)
+			(hide yes)
+			(show_name no)
+			(do_not_autoplace no)
+			(effects
+				(font
+					(size 1.27 1.27)
+				)
+				(justify left)
+			)
+		)
