File: TSC BW 16 V3.1/adc_pins.kicad_sch (KiCad schematic)
At the start: 9 parts, among them J13 Analog Inputs

Commit message: TSC V3 added w5500 v3 rework
Other:
- note added: "ADC PINS / LABELS P14"
Changed lines of the file:
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@@
+	)
+	(rectangle
+		(start 127 160.02)
+		(end 161.29 186.69)
+		(stroke
+			(width 1)
+			(type solid)
+			(color 225 0 0 1)
+		)
+		(fill
+			(type none)
+		)
 	)
 	(rectangle
@@
 		(fill
 			(type none)
+		)
+	)
+	(text "ADC PINS / LABELS P14"
+		(exclude_from_sim no)
+		(at 142.24 155.448 0)
+		(effects
+			(font
+				(size 1.27 1.27)
+			)
 		)
 	)
@@
 	(wire
 		(pts
+			(xy 134.62 163.83) (xy 147.32 163.83)
+		)
+		(stroke
+			(width 0)
+			(type default)
+		)
+	)
+	(wire
+		(pts
 			(xy 185.42 83.82) (xy 203.2 83.82)
 		)
@@
 	(wire
 		(pts
+			(xy 134.62 176.53) (xy 147.32 176.53)
+		)
+		(stroke
+			(width 0)
+			(type default)
+		)
+	)
+	(wire
+		(pts
+			(xy 134.62 181.61) (xy 147.32 181.61)
+		)
+		(stroke
+			(width 0)
+			(type default)
+		)
+	)
+	(wire
+		(pts
 			(xy 113.03 93.98) (xy 113.03 101.6)
 		)
@@
 		(pts
 			(xy 135.89 66.04) (xy 135.89 76.2)
+		)
+		(stroke
+			(width 0)
+			(type default)
+		)
+	)
+	(wire
+		(pts
+			(xy 134.62 170.18) (xy 147.32 170.18)
 		)
 		(stroke
@@
 		)
 	)
-	(label "ANALOG_A4"
-		(at 62.23 90.17 0)
-		(effects
-			(font
-				(size 1.27 1.27)
-			)
-			(justify left bottom)
-		)
-	)
 	(label "ANALOG_A1_INPUT"
 		(at 201.93 81.28 180)
@@
 		)
 	)
-	(label "ANALOG_A2"
-		(at 62.23 82.55 0)
-		(effects
-			(font
-				(size 1.27 1.27)
-			)
-			(justify left bottom)
-		)
-	)
 	(label "ANALOG_A3_INPUT"
 		(at 201.93 86.36 180)
@@
 		)
 	)
+	(label "ANALOG_A2"
+		(at 135.89 170.18 0)
+		(effects
+			(font
+				(size 1.27 1.27)
+			)
+			(justify left bottom)
+		)
+	)
 	(label "ANALOG_A4"
 		(at 161.29 85.09 0)
@@
 		)
 	)
+	(label "ANALOG_A1"
+		(at 135.89 163.83 0)
+		(effects
+			(font
+				(size 1.27 1.27)
+			)
+			(justify left bottom)
+		)
+	)
 	(label "ANALOG_A4_INPUT"
 		(at 201.93 88.9 180)
@@
 	)
 	(label "ANALOG_A3"
-		(at 62.23 86.36 0)
+		(at 135.89 176.53 0)
+		(effects
+			(font
+				(size 1.27 1.27)
+			)
+			(justify left bottom)
+		)
+	)
+	(label "ANALOG_A4"
+		(at 135.89 181.61 0)
 		(effects
 			(font
@@
 		)
 	)
+	(global_label "ANALOG_A2"
+		(shape input)
+		(at 147.32 170.18 0)
+		(fields_autoplaced yes)
+		(effects
+			(font
+				(size 1.27 1.27)
+			)
+			(justify left)
+		)
+		(property "Intersheetrefs" "${INTERSHEET_REFS}"
+			(at 160.7072 170.18 0)
+			(hide yes)
+			(show_name no)
+			(do_not_autoplace no)
+			(effects
+				(font
+					(size 1.27 1.27)
+				)
+				(justify left)
+			)
+		)
+	)
+	(global_label "ANALOG_A3"
+		(shape input)
+		(at 147.32 176.53 0)
+		(fields_autoplaced yes)
+		(effects
+			(font
+				(size 1.27 1.27)
+			)
+			(justify left)
+		)
+		(property "Intersheetrefs" "${INTERSHEET_REFS}"
+			(at 160.7072 176.53 0)
+			(hide yes)
+			(show_name no)
+			(do_not_autoplace no)
+			(effects
+				(font
+					(size 1.27 1.27)
+				)
+				(justify left)
+			)
+		)
+	)
+	(global_label "ANALOG_A1"
+		(shape input)
+		(at 147.32 163.83 0)
+		(fields_autoplaced yes)
+		(effects
+			(font
+				(size 1.27 1.27)
+			)
+			(justify left)
+		)
+		(property "Intersheetrefs" "${INTERSHEET_REFS}"
+			(at 160.7072 163.83 0)
+			(hide yes)
+			(show_name no)
+			(do_not_autoplace no)
+			(effects
+				(font
+					(size 1.27 1.27)
+				)
+				(justify left)
+			)
+		)
+	)
+	(global_label "ANALOG_A4"
+		(shape input)
+		(at 147.32 181.61 0)
+		(fields_autoplaced yes)
+		(effects
+			(font
+				(size 1.27 1.27)
+			)
+			(justify left)
+		)
+		(property "Intersheetrefs" "${INTERSHEET_REFS}"
+			(at 160.7072 181.61 0)
+			(hide yes)
+			(show_name no)
+			(do_not_autoplace no)
+			(effects
+				(font
+					(size 1.27 1.27)
+				)
+				(justify left)
+			)
+		)
+	)

Commit message: WORKING ON IT
Other:
- note added: "Analog Inputs ANALOG_A1 - PIN4 : GPIO4 ANALOG_A2 - PIN6 : GPIO6 ANALOG_A3 - PIN7 : GPIO7 ANALOG_A4 - PIN5 : GPIO5"
Changed lines of the file:
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@@
 	(rectangle
 		(start 127 160.02)
-		(end 161.29 186.69)
+		(end 167.64 195.58)
 		(stroke
 			(width 1)
@@
 		)
 	)
+	(text "Analog Inputs\nANALOG_A1 - PIN4 : GPIO4\nANALOG_A2 - PIN6 : GPIO6\nANALOG_A3 - PIN7 : GPIO7\nANALOG_A4 - PIN5 : GPIO5"
+		(exclude_from_sim no)
+		(at 131.064 188.468 0)
+		(effects
+			(font
+				(size 1.27 1.27)
+				(color 33 191 7 1)
+			)
+			(justify left)
+		)
+	)
