File: TSC BW 16 V3.1/sd_card.kicad_sch (KiCad schematic)
At the start: 2 parts, among them J10 Micro_SD_Card_Det_Hirose_DM3AT

Commit message: WORKING ON IT
Other:
- note added: "SD Card (SPI) MOSI - PIN20 : GPIO12 SCK - PIN21 : GPIO13 MISO - PIN22 : GPIO14 CS - PIN19 : GPIO11 SD-CD - PIN23 : GPIO21"
Changed lines of the file:
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@@
 	(rectangle
 		(start 198.12 85.09)
-		(end 233.68 121.92)
+		(end 233.68 135.89)
 		(stroke
 			(width 1)
@@
 		)
 	)
+	(text "SD Card (SPI)\nMOSI - PIN20 : GPIO12\nSCK - PIN21 : GPIO13\nMISO - PIN22 : GPIO14\nCS - PIN19 : GPIO11\nSD-CD - PIN23 : GPIO21"
+		(exclude_from_sim no)
+		(at 204.978 125.984 0)
+		(effects
+			(font
+				(size 1.27 1.27)
+				(color 33 191 7 1)
+			)
+			(justify left)
+		)
+	)
