File: TSC BW 16 V3.1/untitled.kicad_sch (KiCad schematic)
At the start: 5 parts, among them Q1 BC817

Commit message: WORKING ON IT
Other:
- note added: "BUZZER - PIN25 : GPIO48"
Changed lines of the file:
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@@
+		)
+	)
+	(text "BUZZER - PIN25 : GPIO48 "
+		(exclude_from_sim no)
+		(at 201.676 114.808 0)
+		(effects
+			(font
+				(size 1.27 1.27)
+				(color 33 191 7 1)
+			)
 		)
 	)
