File: TSC BW 16 V3.1/usb_c_to_uart.kicad_sch (KiCad schematic)
At the start: 20 parts, among them J14 USB_C_Receptacle_USB2.0_16P, Q20 SS8050, Q21 SS8050, SW1 SW_Push, SW2 SW_Push, U44 CH340C

Commit message: WORKING ON IT
Other:
- note added: "USB C - UART EN- PIN3 : NO GPIO IO0 - PIN27 : GPIO0 RXD - PIN36/RXD0 : GPIO44,U0RXD TXD - PIN37/ TXD0 : GPIO43,U0TXD"
Changed lines of the file:
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@@
 	)
 	(rectangle
-		(start 218.44 105.41)
-		(end 254 142.24)
+		(start 209.55 105.41)
+		(end 266.7 162.56)
 		(stroke
 			(width 1)
@@
 		)
 	)
+	(text "USB C - UART\nEN- PIN3 : NO GPIO\nIO0 - PIN27 : GPIO0\nRXD - PIN36/RXD0 : GPIO44,U0RXD\nTXD - PIN37/ TXD0 : GPIO43,U0TXD"
+		(exclude_from_sim no)
+		(at 219.71 149.352 0)
+		(effects
+			(font
+				(size 1.27 1.27)
+				(color 33 191 7 1)
+			)
+			(justify left)
+		)
+	)
