File: TSC BW  Proof Of Concept V1/RS485.kicad_sch (KiCad schematic)
At the start: 5 parts, among them J9 BS-12-A1BJ001, U50 AT24CS04-SSHM, U51 DS3231MZ+

Commit message: WORKING ON POC - Proof of concept
Parts:
- removed C45, C46: 0.1uF, Capacitor_SMD:C_1206_3216Metric, symbol Device:C
- removed J9: BS-12-A1BJ001, external_lib:CR1220_HARWIN_S8411-45R, symbol external_lib:CR1220_S8411_45R
- removed U50: AT24CS04-SSHM, Package_SO:SOIC-8_3.9x4.9mm_P1.27mm, symbol Memory_EEPROM:AT24CS04-SSHM
- removed U51: DS3231MZ+, Package_SO:SOIC-8_3.9x4.9mm_P1.27mm, symbol Timer_RTC:DS3231MZ
- added C21: 0.1uF, Capacitor_SMD:C_1206_3216Metric, symbol Device:C
- added D21: SM712_SOT23, Package_TO_SOT_SMD:SOT-23, symbol Diode:SM712_SOT23
- added J12: 691312510002, Connector_Phoenix_MSTB:PhoenixContact_MSTBA_2,5_2-G-5,08_1x02_P5.08mm_Horizontal, symbol pluggable_terminal_connector_2:691312510002
- added R140, R144: 680E, Resistor_SMD:R_1206_3216Metric_Pad1.30x1.75mm_HandSolder, symbol Device:R
- added R141, R143: 10E, Resistor_SMD:R_1206_3216Metric_Pad1.30x1.75mm_HandSolder, symbol Device:R
- added R142: 120E, Resistor_SMD:R_1206_3216Metric_Pad1.30x1.75mm_HandSolder, symbol Device:R
- added U43: SN65HVD75, Package_SO:SOIC-8_3.9x4.9mm_P1.27mm, symbol Interface_UART:SN65HVD11HD
Connections:
- net +3V3: now also C21.2, R144.1, U43.8 (VCC)
- net GND: now also C21.1, D21.3 (common), R140.1, U43.5 (GND)
- new net: R143.1, U43.6 (A)
- new net: R141.1, U43.7 (B)
- new net MCU_EN_RS485: U43.2 (~{RE}), U43.3 (DE)
- new net MCU_Rx_RS485: U43.1 (R)
- new net MCU_Tx_RS485: U43.4 (D)
- new net RS485+: D21.2 (A2), J12.2, R142.2, R143.2, R144.2
- new net RS485-: D21.1 (A1), J12.1, R140.2, R141.2, R142.1
- no-connect marks 3 -> 0
Other:
- note added: "#define RS485_EN 21 void rs485Transmit() { digitalWrite(RS485_EN, HIGH); } void rs485Receive() { digitalWrite(RS485_EN, LOW); } void sendRS485(String msg) { rs485Transmit(); Serial2.print(msg); Serial2.flush(); rs485Receive(); }"
- note added: "RS 485 V1"
- note added: "RS485 TXD - PIN9 : GPIO16 RXD - PIN10 : GPIO17 TXD - PIN23 : GPIO21"
- note removed: "24C04 I2C ADDRESS 0x50 (A1 & A2 -> GND)"
- note removed: "DS3231 I2C ADDRESS 0x68 Fixed"
- note removed: "RTC 2 DS3231MZ+ & 24C04 EEPROM"
- company: (none) -> Tivana Holdings
- title: (none) -> TSC BW 16 V3.1
