File: TSC BW  Proof Of Concept V1/16_digital_inputs.kicad_sch (KiCad schematic)
At the start: 72 parts, among them J5 Terminal Plug, J6 Terminal Plug, U10 PC357C, U11 PC357C, U12 PC357C, U13 PC357C, U14 PC357C, U15 PC357C, U16 PC357C, U17 PC357C, U18 PC357C, U19 PC357C, U20 PCF8574T, U21 PCF8574T, U4 PC357C, U5 PC357C, U6 PC357C, U7 PC357C, U8 PC357C, U9 PC357C

Commit message: WORKING ON POC - Proof of concept
Parts:
- removed H1, H2, H3, H4: MountingHole_Pad, MountingHole:MountingHole_3.2mm_M3_Pad_Via, symbol Mechanical:MountingHole_Pad
- removed J5, J6: Terminal Plug, Connector_Phoenix_MSTB:PhoenixContact_MSTBA_2,5_9-G-5,08_1x09_P5.08mm_Horizontal, symbol pluggable_terminal_connector_9:691312510009
- removed R10, R11, R12, R13, R18, R19, R20, R21, R26, R27, R28, R29, R34, R35, R36, R37: 1k, Resistor_SMD:R_1206_3216Metric_Pad1.30x1.75mm_HandSolder, symbol Device:R
- removed R14, R15, R16, R17, R22, R23, R24, R25, R30, R31, R32, R33, R38, R39, R40, R41: 10k, Resistor_SMD:R_1206_3216Metric_Pad1.30x1.75mm_HandSolder, symbol Device:R
- removed R42, R43, R44, R45, R46, R47, R48, R49, R50, R51, R52, R53, R54, R55, R56, R57: 4.7k, Resistor_SMD:R_1206_3216Metric_Pad1.30x1.75mm_HandSolder, symbol Device:R
- removed U10, U11, U12, U13, U14, U15, U16, U17, U18, U19, U4, U5, U6, U7, U8, U9: PC357C, Package_SO:SO-4_4.4x4.3mm_P2.54mm, symbol Lucasian:PC357C
- removed U20, U21: PCF8574T, Package_SO:SOIC-16W_7.5x10.3mm_P1.27mm, symbol Interface_Expansion:PCF8574T
Connections:
- no-connect marks 2 -> 0
Other:
- note removed: "16 DIGITAL ISOLATED INPUTS"
- note removed: "GLOBAL PINS / LABELS"
- note removed: "INPUTS 1"
- note removed: "INPUTS 2"
- note removed: "Input Terminal Block 1"
- note removed: "Input Terminal Block 2"
- note removed: "PCF8574 I2C ADDRESS INPUT 2: 0X21"
- note removed: "PCF8574 I2C ADDRESS Input 1: 0X20"
- company: Tivana Holdings -> (none)
- title: TSC BW 16 V3.1 -> (none)
