File: TSC BW  Proof Of Concept V1/16_digital_outputs.kicad_sch (KiCad schematic)
At the start: 120 parts, among them J7 Terminal Plug, J8 Terminal Plug, Q10 NCE60P10K, Q11 NCE60P10K, Q12 NCE60P10K, Q13 NCE60P10K, Q14 NCE60P10K, Q15 NCE60P10K, Q16 NCE60P10K, Q17 NCE60P10K, Q18 NCE60P10K, Q19 NCE60P10K, Q4 NCE60P10K, Q5 NCE60P10K, Q6 NCE60P10K, Q7 NCE60P10K, Q8 NCE60P10K, Q9 NCE60P10K, U22 PC357C, U23 PC357C, U24 PC357C, U25 PC357C, U26 PC357C, U27 PC357C, U28 PC357C, U29 PC357C, U30 PC357C, U31 PC357C, U32 PC357C, U33 PC357C, U34 PC357C, U35 PC357C, U36 PC357C, U37 PC357C, U38 PCF8574T, U39 PCF8574T

Commit message: WORKING ON POC - Proof of concept
Parts:
- removed D10, D11, D12, D13, D14, D15, D16, D17, D18, D19, D20, D5, D6, D7, D8, D9: IR26-21C_L110_TR8, LED_SMD:LED_1206_3216Metric, symbol LED:IR26-21C_L110_TR8
- removed J7, J8: Terminal Plug, Connector_Phoenix_MSTB:PhoenixContact_MSTBA_2,5_9-G-5,08_1x09_P5.08mm_Horizontal, symbol pluggable_terminal_connector_9:691312510009
- removed Q10, Q11, Q12, Q13, Q14, Q15, Q16, Q17, Q18, Q19, Q4, Q5, Q6, Q7, Q8, Q9: NCE60P10K, Package_TO_SOT_SMD:TO-252-2, symbol Transistor_FET:SUD08P06-155L
- removed R100, R110, R112, R114, R116, R62, R64, R66, R68, R78, R80, R82, R84, R94, R96, R98: 1k, Resistor_SMD:R_1206_3216Metric_Pad1.30x1.75mm_HandSolder, symbol Device:R
- removed R101, R111, R113, R115, R117, R63, R65, R67, R69, R79, R81, R83, R85, R95, R97, R99: 8.2k, Resistor_SMD:R_1206_3216Metric_Pad1.30x1.75mm_HandSolder, symbol Device:R
- removed R102, R103, R104, R105, R118, R119, R120, R121, R70, R71, R72, R73, R86, R87, R88, R89: 5.1K, Resistor_SMD:R_1206_3216Metric_Pad1.30x1.75mm_HandSolder, symbol Device:R
- removed R106, R107, R108, R109, R58, R59, R60, R61, R74, R75, R76, R77, R90, R91, R92, R93: 4.7K, Resistor_SMD:R_1206_3216Metric_Pad1.30x1.75mm_HandSolder, symbol Device:R
- removed RN1, RN2, RN3, RN4: resister_array_4_10k_CAY16-103J4LF, Resistor_SMD:R_Array_Convex_4x0603, symbol CAY16-103J4LF:resister_array_4_10k_CAY16-103J4LF
- removed U22, U23, U24, U25, U26, U27, U28, U29, U30, U31, U32, U33, U34, U35, U36, U37: PC357C, Package_SO:SO-4_4.4x4.3mm_P2.54mm, symbol Lucasian:PC357C
- removed U38, U39: PCF8574T, Package_SO:SOIC-16W_7.5x10.3mm_P1.27mm, symbol Interface_Expansion:PCF8574T
Connections:
- no-connect marks 2 -> 0
Other:
- note removed: "16 ISOLATED OUTPUTS"
- note removed: "GLOBAL PINS / LABELS"
- note removed: "OUTPUTS 1"
- note removed: "OUTPUTS 2"
- note removed: "Output Terminal Block 1"
- note removed: "Output Terminal Block 2"
- note removed: "PCF Pull Up Resistors"
- note removed: "PCF8574 I2C ADDRESS OUTPUT 1: 0X22"
- note removed: "PCF8575 I2C ADDRESS OUTPUT 2: 0X23"
- company: Tivana Holdings -> (none)
- title: TSC BW 16 V3.1 -> (none)
