File: TSC BW  Proof Of Concept V1/TSC BW 16 V3 POC.kicad_sch (KiCad schematic)
At the start: 0 parts

Commit message: WORKING ON POC - Proof of concept
Other:
- sheet 16 DIGITAL INPUTS renamed 8 DIGITAL INPUTS
- sheet 16 DIGITAL OUTPUTS renamed 8 DIGITAL OUTPUTS
- sheet 8 DIGITAL INPUTS: file 16_digital_inputs.kicad_sch -> 8_digital_inputs.kicad_sch
- sheet 8 DIGITAL OUTPUTS: file 16_digital_outputs.kicad_sch -> 8_digital_outputs.kicad_sch
Changed lines of the file:
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@@
 		)
 		(instances
-			(project "TSC BW 16 V3"
+			(project "TSC BW 16 V3 POC"
 				(path "/65a0f6c1-6a57-4cd2-a77c-79691e6171da"
 					(page "8")
@@
 		)
 		(instances
-			(project "TSC BW 16 V3"
+			(project "TSC BW 16 V3 POC"
 				(path "/65a0f6c1-6a57-4cd2-a77c-79691e6171da"
 					(page "14")
@@
 		)
 		(fill
-			(color 43 255 0 1)
+			(color 255 240 4 1)
 		)
 		(property "Sheetname" "RS485 v2"
@@
 		)
 		(instances
-			(project "TSC BW 16 V3"
+			(project "TSC BW 16 V3 POC"
 				(path "/65a0f6c1-6a57-4cd2-a77c-79691e6171da"
 					(page "10")
@@
 			(color 7 255 1 1)
 		)
-		(property "Sheetname" "16 DIGITAL INPUTS"
+		(property "Sheetname" "8 DIGITAL INPUTS"
 			(at 19.05 55.1684 0)
 			(show_name no)
@@
 			)
 		)
-		(property "Sheetfile" "16_digital_inputs.kicad_sch"
+		(property "Sheetfile" "8_digital_inputs.kicad_sch"
 			(at 19.05 78.0546 0)
 			(show_name no)
@@
 		)
 		(instances
-			(project "TSC BW 16 V3"
+			(project "TSC BW 16 V3 POC"
 				(path "/65a0f6c1-6a57-4cd2-a77c-79691e6171da"
 					(page "4")
@@
 			(color 4 255 0 1)
 		)
-		(property "Sheetname" "16 DIGITAL OUTPUTS"
+		(property "Sheetname" "8 DIGITAL OUTPUTS"
 			(at 20.32 88.1884 0)
 			(show_name no)
@@
 			)
 		)
-		(property "Sheetfile" "16_digital_outputs.kicad_sch"
+		(property "Sheetfile" "8_digital_outputs.kicad_sch"
 			(at 20.32 109.8046 0)
 			(show_name no)
@@
 		)
 		(instances
-			(project "TSC BW 16 V3"
+			(project "TSC BW 16 V3 POC"
 				(path "/65a0f6c1-6a57-4cd2-a77c-79691e6171da"
 					(page "5")
@@
 		)
 		(instances
-			(project "TSC BW 16 V3"
+			(project "TSC BW 16 V3 POC"
 				(path "/65a0f6c1-6a57-4cd2-a77c-79691e6171da"
 					(page "13")
@@
 		)
 		(instances
-			(project "TSC BW 16 V3"
+			(project "TSC BW 16 V3 POC"
 				(path "/65a0f6c1-6a57-4cd2-a77c-79691e6171da"
 					(page "9")
@@
 		)
 		(instances
-			(project "TSC BW 16 V3"
+			(project "TSC BW 16 V3 POC"
 				(path "/65a0f6c1-6a57-4cd2-a77c-79691e6171da"
 					(page "2")
@@
 		)
 		(instances
-			(project "TSC BW 16 V3"
+			(project "TSC BW 16 V3 POC"
 				(path "/65a0f6c1-6a57-4cd2-a77c-79691e6171da"
 					(page "12")
@@
 		)
 		(instances
-			(project "TSC BW 16 V3"
+			(project "TSC BW 16 V3 POC"
 				(path "/65a0f6c1-6a57-4cd2-a77c-79691e6171da"
 					(page "7")
@@
 		)
 		(instances
-			(project "TSC BW 16 V3"
+			(project "TSC BW 16 V3 POC"
 				(path "/65a0f6c1-6a57-4cd2-a77c-79691e6171da"
 					(page "11")
@@
 		)
 		(instances
-			(project "TSC BW 16 V3"
+			(project "TSC BW 16 V3 POC"
 				(path "/65a0f6c1-6a57-4cd2-a77c-79691e6171da"
 					(page "16")
@@
 		)
 		(instances
-			(project "TSC BW 16 V3"
+			(project "TSC BW 16 V3 POC"
 				(path "/65a0f6c1-6a57-4cd2-a77c-79691e6171da"
 					(page "15")
@@
 		)
 		(instances
-			(project "TSC BW 16 V3"
+			(project "TSC BW 16 V3 POC"
 				(path "/65a0f6c1-6a57-4cd2-a77c-79691e6171da"
 					(page "6")
@@
 		)
 		(instances
-			(project "TSC BW 16 V3"
+			(project "TSC BW 16 V3 POC"
 				(path "/65a0f6c1-6a57-4cd2-a77c-79691e6171da"
 					(page "3")
@@
 		)
 		(instances
-			(project "TSC BW 16 V3"
+			(project "TSC BW 16 V3 POC"
 				(path "/65a0f6c1-6a57-4cd2-a77c-79691e6171da"
 					(page "17")

Commit message: WORKING ON POC - Proof of concept
Other:
- removed sheet ETHERNET
- removed sheet Ethernet W5500
- removed sheet External Connections
- removed sheet RS485 v1
- removed sheet RTC2
