File: TSC BW  Proof Of Concept V1/RS485 v2.kicad_sch (KiCad schematic)
At the start: 20 parts, among them J15 691312510002, J17 691312510002, U47 MAX13487EESA, U48 MAX13487EESA

Commit message: WORKING ON POC - Proof of concept
Parts:
- removed C26: 10uF, Capacitor_SMD:C_1206_3216Metric, symbol Device:C
- removed C27: 100nF, Capacitor_SMD:C_1206_3216Metric, symbol Device:C
- removed D26, D27: D_TVS: SMBJ6.8CA, symbol Device:D_TVS
- removed F1, F2: PPTC 60V/0.1A, symbol Device:Polyfuse
- removed J15: 691312510002, Connector_Phoenix_MSTB:PhoenixContact_MSTBA_2,5_2-G-5,08_1x02_P5.08mm_Horizontal, symbol pluggable_terminal_connector_2:691312510002
- removed R161, R162: 680E, Resistor_SMD:R_1206_3216Metric_Pad1.30x1.75mm_HandSolder, symbol Device:R
- removed R163: 120R, Resistor_SMD:R_1206_3216Metric_Pad1.30x1.75mm_HandSolder, symbol Device:R
- removed U47: MAX13487EESA, Package_SO:SOIC-8_3.9x4.9mm_P1.27mm, symbol Interface_UART:SN65HVD11HD
- D28, D29: footprint (none) -> Diode_SMD:D_SMB
- F3, F4: value PPTC 60V/0.1A -> PPTC 60V/10R; footprint (none) -> Fuse:Fuse_1206_3216Metric

Commit message: WORKING ON POC - Proof of concept
Parts:
- added JP7: SolderJumper_2_Open, Jumper:SolderJumper-2_P1.3mm_Open_RoundedPad1.0x1.5mm, symbol Jumper:SolderJumper_2_Open
Connections:
- net +3V3: now also JP7.1 (A); no longer U48.8 (VCC)
- new net: JP7.2 (B), U48.8 (VCC)
Changed lines of the file:
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@@
+	(wire
+		(pts
+			(xy 99.06 54.61) (xy 99.06 59.69)
+		)
+		(stroke
+			(width 0)
+			(type default)
+		)
+	)
 	(wire
 		(pts
@@
 	(wire
 		(pts
-			(xy 99.06 48.26) (xy 99.06 59.69)
+			(xy 99.06 36.83) (xy 99.06 44.45)
 		)
 		(stroke
@@
 	(symbol
 		(lib_id "power:+3V3")
-		(at 99.06 48.26 0)
+		(at 99.06 36.83 0)
 		(unit 1)
 		(body_style 1)
@@
 		(fields_autoplaced yes)
 		(property "Reference" "#PWR0233"
-			(at 99.06 52.07 0)
+			(at 99.06 40.64 0)
 			(hide yes)
 			(show_name no)
@@
 		)
 		(property "Value" "+3V3"
-			(at 99.06 43.18 0)
+			(at 99.06 31.75 0)
 			(show_name no)
 			(do_not_autoplace no)
@@
 		)
 		(property "Footprint" ""
-			(at 99.06 48.26 0)
+			(at 99.06 36.83 0)
 			(hide yes)
 			(show_name no)
@@
 		)
 		(property "Datasheet" ""
-			(at 99.06 48.26 0)
+			(at 99.06 36.83 0)
 			(hide yes)
 			(show_name no)
@@
 		)
 		(property "Description" "Power symbol creates a global label with name \"+3V3\""
-			(at 99.06 48.26 0)
+			(at 99.06 36.83 0)
 			(hide yes)
 			(show_name no)
@@
 					(unit 1)
 				)
+			)
+		)
+	)
+	(symbol
+		(lib_id "Jumper:SolderJumper_2_Open")
+		(at 99.06 49.53 270)
+		(unit 1)
+		(body_style 1)
+		(exclude_from_sim no)
+		(in_bom no)
+		(on_board yes)
+		(in_pos_files yes)
+		(dnp no)
+		(fields_autoplaced yes)
+		(property "Reference" "JP7"
+			(at 101.6 49.5299 90)
+			(show_name no)
+			(do_not_autoplace no)
+			(effects
+				(font
+					(size 1.27 1.27)
+				)
+				(justify left)
+			)
+		)
+		(property "Value" "SolderJumper_2_Open"
+			(at 102.87 49.53 0)
+			(hide yes)
+			(show_name no)
+			(do_not_autoplace no)
+			(effects
+				(font
+					(size 1.27 1.27)
+				)
+			)
+		)
+		(property "Footprint" "Jumper:SolderJumper-2_P1.3mm_Open_RoundedPad1.0x1.5mm"
+			(at 99.06 49.53 0)
+			(hide yes)
+			(show_name no)
+			(do_not_autoplace no)
+			(effects
+				(font
+					(size 1.27 1.27)
+				)
+			)
+		)
+		(property "Datasheet" ""
+			(at 91.44 49.53 0)
+			(hide yes)
+			(show_name no)
+			(do_not_autoplace no)
+			(effects
+				(font
+					(size 1.27 1.27)
+				)
+			)
+		)
+		(property "Description" "Solder Jumper, 2-pole, open"
+			(at 93.98 49.53 0)
+			(hide yes)
+			(show_name no)
+			(do_not_autoplace no)
+			(effects
+				(font
+					(size 1.27 1.27)
+				)
+			)
+		)
+		(pin "2"
+		)
+		(pin "1"
+		)
+		(instances
+			(project "TSC BW 16 V3 POC"
+				(path "/65a0f6c1-6a57-4cd2-a77c-79691e6171da/40ee65e9-2fd8-4eed-8511-b217a3b2d635"
+					(reference "JP7")
+					(unit 1)
+				)
