File: TSC BW  Proof Of Concept V1/adc_pins.kicad_sch (KiCad schematic)
At the start: 9 parts, among them J13 Analog Inputs

Commit message: WORKING ON POC - Proof of concept
Parts:
- added C26, C27, C28, C29: 10pF, Capacitor_SMD:C_1206_3216Metric, symbol Device:C
Connections:
- net ANALOG_A1: now also C26.2
- net ANALOG_A2: now also C27.2
- net ANALOG_A3: now also C28.2
- net ANALOG_A4: now also C29.2
- net GND: now also C26.1, C27.1, C28.1, C29.1
