File: TSC BW  Proof Of Concept V1/rtc.kicad_sch (KiCad schematic)
At the start: 5 parts, among them J9 BS-12-A1BJ001, U50 AT24CS04-SSHM, U51 DS3231MZ+

Commit message: WORKING ON POC - Proof of concept
Parts:
- removed C45, C46: 0.1uF, Capacitor_SMD:C_1206_3216Metric, symbol Device:C
- removed J9: BS-12-A1BJ001, external_lib:CR1220_HARWIN_S8411-45R, symbol external_lib:CR1220_S8411_45R
- removed U50: AT24CS04-SSHM, Package_SO:SOIC-8_3.9x4.9mm_P1.27mm, symbol Memory_EEPROM:AT24CS04-SSHM
- removed U51: DS3231MZ+, Package_SO:SOIC-8_3.9x4.9mm_P1.27mm, symbol Timer_RTC:DS3231MZ
- added C43, C44: 0.1uF, Capacitor_SMD:C_1206_3216Metric, symbol Device:C
- added J2: CR1220_S8411_45R, external_lib:CR1220_HARWIN_S8411-45R, symbol external_lib:CR1220_S8411_45R
- added U40: AT24CS04-SSHM, Package_SO:SOIC-8_3.9x4.9mm_P1.27mm, symbol Memory_EEPROM:AT24CS04-SSHM
- added U41: DS3231MZ, Package_SO:SOIC-8_3.9x4.9mm_P1.27mm, symbol Timer_RTC:DS3231MZ
Connections:
- net +3V3: now also C43.1, C44.1, U40.8 (VCC), U41.2 (VCC)
- net GND: now also C43.2, C44.2, J2.N, U40.2 (A1), U40.3 (A2), U40.4 (GND), U40.7 (WP), U41.5 (GND)
- net SCL: now also U40.6 (SCL), U41.8 (SCL)
- net SDA: now also U40.5 (SDA), U41.7 (SDA)
- new net: J2.P, U41.6 (VBAT)
Other:
- note added: "RTC DS3231 & 24C04 EEPROM"
- note removed: "RTC 2 DS3231MZ+ & 24C04 EEPROM"
- company: (none) -> Tivana Holdings
- title: (none) -> TSC BW 16 V3.1

Commit message: WORKING ON POC - Proof of concept
Parts:
- added JP2: SolderJumper_2_Open, Jumper:SolderJumper-2_P1.3mm_Open_RoundedPad1.0x1.5mm, symbol Jumper:SolderJumper_2_Open
Connections:
- net +3V3: now also JP2.2 (B); no longer C43.1, C44.1, U40.8 (VCC), U41.2 (VCC)
- new net: C43.1, C44.1, JP2.1 (A), U40.8 (VCC), U41.2 (VCC)
Changed lines of the file:
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@@
 	(text "       RTC\nDS3231 & 24C04 EEPROM"
 		(exclude_from_sim no)
-		(at 124.206 51.054 0)
+		(at 124.968 31.496 0)
 		(effects
 			(font
@@
 		(color 0 0 0 0)
 	)
+	(junction
+		(at 99.06 71.12)
+		(diameter 0)
+		(color 0 0 0 0)
+	)
 	(no_connect
 		(at 160.02 93.98)
@@
 	(wire
 		(pts
+			(xy 152.4 52.07) (xy 121.92 52.07)
+		)
+		(stroke
+			(width 0)
+			(type default)
+		)
+	)
+	(wire
+		(pts
+			(xy 99.06 71.12) (xy 99.06 77.47)
+		)
+		(stroke
+			(width 0)
+			(type default)
+		)
+	)
+	(wire
+		(pts
 			(xy 99.06 77.47) (xy 99.06 78.74)
 		)
@@
 	(wire
 		(pts
-			(xy 99.06 74.93) (xy 99.06 77.47)
+			(xy 99.06 50.8) (xy 99.06 53.34)
 		)
 		(stroke
@@
 	(wire
 		(pts
+			(xy 121.92 71.12) (xy 99.06 71.12)
+		)
+		(stroke
+			(width 0)
+			(type default)
+		)
+	)
+	(wire
+		(pts
+			(xy 99.06 63.5) (xy 99.06 71.12)
+		)
+		(stroke
+			(width 0)
+			(type default)
+		)
+	)
+	(wire
+		(pts
 			(xy 144.78 66.04) (xy 144.78 69.85)
 		)
@@
 	(wire
 		(pts
-			(xy 152.4 66.04) (xy 152.4 85.09)
+			(xy 152.4 52.07) (xy 152.4 85.09)
 		)
 		(stroke
@@
 		(pts
 			(xy 163.83 85.09) (xy 166.37 85.09)
+		)
+		(stroke
+			(width 0)
+			(type default)
+		)
+	)
+	(wire
+		(pts
+			(xy 121.92 52.07) (xy 121.92 71.12)
 		)
 		(stroke
@@
 	)
 	(symbol
-		(lib_id "power:+3V3")
-		(at 152.4 66.04 0)
-		(unit 1)
-		(body_style 1)
-		(exclude_from_sim no)
-		(in_bom yes)
-		(on_board yes)
-		(in_pos_files yes)
-		(dnp no)
-		(property "Reference" "#PWR0176"
-			(at 152.4 69.85 0)
-			(hide yes)
-			(show_name no)
-			(do_not_autoplace no)
-			(effects
-				(font
-					(size 1.27 1.27)
-				)
-			)
-		)
-		(property "Value" "+3V3"
-			(at 154.686 68.072 90)
-			(show_name no)
-			(do_not_autoplace no)
-			(effects
-				(font
-					(size 1.27 1.27)
-				)
-			)
-		)
-		(property "Footprint" ""
-			(at 152.4 66.04 0)
-			(hide yes)
-			(show_name no)
-			(do_not_autoplace no)
-			(effects
-				(font
-					(size 1.27 1.27)
-				)
-			)
-		)
-		(property "Datasheet" ""
-			(at 152.4 66.04 0)
-			(hide yes)
-			(show_name no)
-			(do_not_autoplace no)
-			(effects
-				(font
-					(size 1.27 1.27)
-				)
-			)
-		)
-		(property "Description" "Power symbol creates a global label with name \"+3V3\""
-			(at 152.4 66.04 0)
-			(hide yes)
-			(show_name no)
-			(do_not_autoplace no)
-			(effects
-				(font
-					(size 1.27 1.27)
-				)
-			)
-		)
-		(pin "1"
-		)
-		(instances
-			(project "TSC BW 16 V3 POC"
-				(path "/65a0f6c1-6a57-4cd2-a77c-79691e6171da/f360778a-4100-4e67-bb28-4591c77fa6f9"
-					(reference "#PWR0176")
-					(unit 1)
-				)
-			)
-		)
-	)
-	(symbol
 		(lib_id "Device:C")
 		(at 87.63 77.47 270)
@@
 	)
 	(symbol
+		(lib_id "Jumper:SolderJumper_2_Open")
+		(at 99.06 58.42 90)
+		(unit 1)
+		(body_style 1)
+		(exclude_from_sim no)
+		(in_bom no)
+		(on_board yes)
+		(in_pos_files yes)
+		(dnp no)
+		(fields_autoplaced yes)
+		(property "Reference" "JP2"
+			(at 101.6 58.4199 90)
+			(show_name no)
+			(do_not_autoplace no)
+			(effects
+				(font
+					(size 1.27 1.27)
+				)
+				(justify right)
+			)
+		)
+		(property "Value" "SolderJumper_2_Open"
+			(at 95.25 58.42 0)
+			(hide yes)
+			(show_name no)
+			(do_not_autoplace no)
+			(effects
+				(font
+					(size 1.27 1.27)
+				)
+			)
+		)
+		(property "Footprint" "Jumper:SolderJumper-2_P1.3mm_Open_RoundedPad1.0x1.5mm"
+			(at 99.06 58.42 0)
+			(hide yes)
+			(show_name no)
+			(do_not_autoplace no)
+			(effects
+				(font
+					(size 1.27 1.27)
+				)
+			)
+		)
+		(property "Datasheet" ""
+			(at 106.68 58.42 0)
+			(hide yes)
+			(show_name no)
+			(do_not_autoplace no)
+			(effects
+				(font
+					(size 1.27 1.27)
+				)
+			)
+		)
+		(property "Description" "Solder Jumper, 2-pole, open"
+			(at 104.14 58.42 0)
+			(hide yes)
+			(show_name no)
+			(do_not_autoplace no)
+			(effects
+				(font
+					(size 1.27 1.27)
+				)
+			)
+		)
+		(pin "2"
+		)
+		(pin "1"
+		)
+		(instances
+			(project "TSC BW 16 V3 POC"
+				(path "/65a0f6c1-6a57-4cd2-a77c-79691e6171da/f360778a-4100-4e67-bb28-4591c77fa6f9"
+					(reference "JP2")
+					(unit 1)
+				)
+			)
+		)
+	)
+	(symbol
 		(lib_id "Memory_EEPROM:AT24CS04-SSHM")
 		(at 99.06 86.36 0)
@@
 	(symbol
 		(lib_id "power:+3V3")
-		(at 99.06 74.93 0)
+		(at 99.06 50.8 0)
 		(unit 1)
 		(body_style 1)
@@
 		(fields_autoplaced yes)
 		(property "Reference" "#PWR0177"
-			(at 99.06 78.74 0)
+			(at 99.06 54.61 0)
 			(hide yes)
 			(show_name no)
@@
 		)
 		(property "Value" "+3V3"
-			(at 99.06 69.85 0)
+			(at 99.06 45.72 0)
 			(show_name no)
 			(do_not_autoplace no)
@@
 		)
 		(property "Footprint" ""
-			(at 99.06 74.93 0)
+			(at 99.06 50.8 0)
 			(hide yes)
 			(show_name no)
@@
 		)
 		(property "Datasheet" ""
-			(at 99.06 74.93 0)
+			(at 99.06 50.8 0)
 			(hide yes)
 			(show_name no)
@@
 		)
 		(property "Description" "Power symbol creates a global label with name \"+3V3\""
-			(at 99.06 74.93 0)
-			(hide yes)
-			(show_name no)
+			(at 99.06 50.8 0)
+			(hide yes)
+			(show_name no)

Commit message: WORKING ON POC - Proof of concept
Parts:
- J2: footprint external_lib:CR1220_HARWIN_S8411-45R -> Battery:BatteryHolder_Keystone_500
Connections:
- net GND: now also J2.2; no longer J2.N
- net at U41.6 (VBAT): now also J2.1; no longer J2.P
Changed lines of the file:
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@@
+	(wire
+		(pts
+			(xy 144.78 85.09) (xy 144.78 88.9)
+		)
+		(stroke
+			(width 0)
+			(type default)
+		)
+	)
 	(wire
 		(pts
@@
 		(pts
 			(xy 109.22 83.82) (xy 119.38 83.82)
-		)
-		(stroke
-			(width 0)
-			(type default)
-		)
-	)
-	(wire
-		(pts
-			(xy 144.78 85.09) (xy 144.78 88.9)
 		)
 		(stroke
@@
 			)
 		)
-		(property "Footprint" "external_lib:CR1220_HARWIN_S8411-45R"
-			(at 144.78 77.47 0)
+		(property "Footprint" "Battery:BatteryHolder_Keystone_500"
+			(at 135.89 75.946 0)
 			(hide yes)
 			(show_name no)
@@
 		)
 		(property "Description" "Coin Cell Battery Retainer, Horizontal SMT, for CR1220 Coin Cell Batteries, Tape & Reeled"
-			(at 144.78 77.47 0)
+			(at 158.242 75.946 0)
 			(hide yes)
 			(show_name no)
@@
 		)
 		(property "MAXIMUM_PACKAGE_HEIGHT" "4.25mm"
-			(at 144.78 77.47 0)
+			(at 147.828 63.5 0)
 			(hide yes)
 			(show_name no)
@@
 		)
 		(property "Package" "None"
-			(at 144.78 77.47 0)
+			(at 147.574 76.962 0)
 			(hide yes)
 			(show_name no)
@@
 		)
 		(property "Price" "None"
-			(at 144.78 77.47 0)
+			(at 140.462 64.516 0)
 			(hide yes)
 			(show_name no)
@@
 		)
 		(property "Check_prices" "https://www.snapeda.com/parts/S8411-45R/Harwin/view-part/?ref=eda"
-			(at 144.78 77.47 0)
+			(at 157.226 74.168 0)
 			(hide yes)
 			(show_name no)
@@
 		)
 		(property "STANDARD" "Manufacturer Recommendations"
-			(at 144.78 77.47 0)
+			(at 154.94 75.946 0)
 			(hide yes)
 			(show_name no)
@@
 		)
 		(property "SnapEDA_Link" "https://www.snapeda.com/parts/S8411-45R/Harwin/view-part/?ref=snap"
-			(at 144.78 77.47 0)
+			(at 151.892 78.74 0)
 			(hide yes)
 			(show_name no)
@@
 		)
 		(property "MP" "S8411-45R"
-			(at 144.78 77.47 0)
+			(at 147.32 77.216 0)
 			(hide yes)
 			(show_name no)
@@
 		)
 		(property "Availability" "In Stock"
-			(at 144.78 77.47 0)
+			(at 143.002 62.23 0)
 			(hide yes)
 			(show_name no)
@@
 		)
 		(property "MANUFACTURER" "Harwin"
-			(at 144.78 77.47 0)
-			(hide yes)
-			(show_name no)
-			(do_not_autoplace no)
-			(effects
-				(font
-					(size 1.27 1.27)
-				)
-				(justify bottom)
-			)
-		)
-		(pin "P"
-		)
-		(pin "N"
+			(at 148.844 76.962 0)
+			(hide yes)
+			(show_name no)
+			(do_not_autoplace no)
+			(effects
+				(font
+					(size 1.27 1.27)
+				)
+				(justify bottom)
+			)
+		)
+		(pin "2"
+		)
+		(pin "1"
 		)
 		(instances
