File: TSC BW  Proof Of Concept V1/8_digital_outputs.kicad_sch (KiCad schematic)
At the start: 60 parts, among them J7 Terminal Plug, Q10 NCE60P10K, Q11 NCE60P10K, Q14 NCE60P10K, Q15 NCE60P10K, Q18 NCE60P10K, Q19 NCE60P10K, Q6 NCE60P10K, Q7 NCE60P10K, U24 PC357C, U25 PC357C, U28 PC357C, U29 PC357C, U32 PC357C, U33 PC357C, U36 PC357C, U37 PC357C, U38 PCF8574T

Commit message: WORKING ON POC - Proof of concept
Parts:
- R104, R105, R120, R121, R72, R73, R88, R89: value 5.1K -> 10k
- R115, R117, R67, R69, R83, R85, R99: value 8.2k -> 470R
- RN1, RN2: footprint Resistor_SMD:R_Array_Convex_4x0603 -> Resistor_SMD:R_Array_Convex_4x1206
Other:
- note added: "8 ISOLATED OUTPUTS"
- note removed: "16 ISOLATED OUTPUTS"
Changed lines of the file:
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@@
 		)
 	)
-	(text "16 ISOLATED OUTPUTS"
+	(text "8 ISOLATED OUTPUTS"
 		(exclude_from_sim no)
 		(at 219.71 44.704 0)
@@
 	)
 	(junction
-		(at 276.86 237.49)
+		(at 90.17 60.96)
 		(diameter 0)
 		(color 0 0 0 0)
 	)
 	(junction
-		(at 281.94 237.49)
+		(at 92.71 156.21)
 		(diameter 0)
 		(color 0 0 0 0)
 	)
 	(junction
-		(at 90.17 60.96)
+		(at 276.86 237.49)
 		(diameter 0)
 		(color 0 0 0 0)
 	)
 	(junction
-		(at 92.71 156.21)
+		(at 77.47 133.35)
 		(diameter 0)
 		(color 0 0 0 0)
 	)
 	(junction
-		(at 77.47 133.35)
+		(at 132.08 237.49)
 		(diameter 0)
 		(color 0 0 0 0)
 	)
 	(junction
-		(at 132.08 237.49)
+		(at 281.94 237.49)
 		(diameter 0)
 		(color 0 0 0 0)
 	)
 	(junction
-		(at 271.78 237.49)
+		(at 91.44 124.46)
 		(diameter 0)
 		(color 0 0 0 0)
 	)
 	(junction
-		(at 91.44 124.46)
+		(at 271.78 237.49)
 		(diameter 0)
 		(color 0 0 0 0)
@@
 			)
 		)
-		(property "Value" "8.2k"
+		(property "Value" "470R"
 			(at 73.914 133.35 90)
 			(show_name no)
@@
 			)
 		)
-		(property "Value" "8.2k"
+		(property "Value" "470R"
 			(at 75.184 165.1 90)
 			(show_name no)
@@
 			)
 		)
-		(property "Value" "8.2k"
+		(property "Value" "470R"
 			(at 72.644 67.31 90)
 			(show_name no)
@@
 			)
 		)
-		(property "Value" "5.1K"
+		(property "Value" "10k"
 			(at 300.99 70.866 90)
 			(show_name no)
@@
 			)
 		)
-		(property "Value" "5.1K"
+		(property "Value" "10k"
 			(at 302.26 136.906 90)
 			(show_name no)
@@
 			)
 		)
-		(property "Value" "8.2k"
+		(property "Value" "470R"
 			(at 299.974 162.56 90)
 			(show_name no)
@@
 			)
 		)
-		(property "Value" "8.2k"
+		(property "Value" "470R"
 			(at 297.434 64.77 90)
 			(show_name no)
@@
 			)
 		)
-		(property "Value" "5.1K"
+		(property "Value" "10k"
 			(at 76.2 73.406 90)
 			(show_name no)
@@
 			)
 		)
-		(property "Value" "5.1K"
+		(property "Value" "10k"
 			(at 78.74 171.196 90)
 			(show_name no)
@@
 			)
 		)
-		(property "Value" "8.2k"
+		(property "Value" "470R"
 			(at 73.914 99.06 90)
 			(show_name no)
@@
 			)
 		)
-		(property "Value" "5.1K"
+		(property "Value" "10k"
 			(at 77.47 105.156 90)
 			(show_name no)
@@
 	)
 	(symbol
+		(lib_name "SUD08P06-155L_1")
 		(lib_id "Transistor_FET:SUD08P06-155L")
 		(at 88.9 99.06 0)
@@
 		(in_pos_files yes)
 		(dnp no)
-		(fields_autoplaced yes)
 		(property "Reference" "RN2"
 			(at 288.29 227.3299 90)
@@
 		)
 		(property "Value" "resister_array_4_10k_CAY16-103J4LF"
-			(at 288.29 228.5999 90)
-			(hide yes)
+			(at 288.544 230.632 90)
 			(show_name no)
 			(do_not_autoplace no)
@@
 			)
 		)
-		(property "Footprint" "Resistor_SMD:R_Array_Convex_4x0603"
+		(property "Footprint" "Resistor_SMD:R_Array_Convex_4x1206"
 			(at 274.32 227.33 0)
 			(hide yes)
@@
 			)
 		)
-		(property "Value" "5.1K"
+		(property "Value" "10k"
 			(at 303.53 168.656 90)
 			(show_name no)
@@
 			)
 		)
-		(property "Value" "5.1K"
+		(property "Value" "10k"
 			(at 302.26 102.616 90)
 			(show_name no)
@@
 			)
 		)
-		(property "Value" "8.2k"
+		(property "Value" "470R"
 			(at 298.704 96.52 90)
 			(show_name no)
@@
 		)
 		(property "Value" "8.2k"
-			(at 298.704 130.81 90)
+			(at 298.704 11.938 90)
 			(show_name no)
 			(do_not_autoplace no)
@@
 			)
 		)
-		(property "Value" "5.1K"
+		(property "Value" "10k"
 			(at 77.47 139.446 90)
 			(show_name no)
@@
 		(in_pos_files yes)
 		(dnp no)
-		(fields_autoplaced yes)
 		(property "Reference" "RN1"
 			(at 148.59 227.3299 90)
@@
 		)
 		(property "Value" "resister_array_4_10k_CAY16-103J4LF"
-			(at 148.59 228.5999 90)
-			(hide yes)
+			(at 148.336 229.616 90)
 			(show_name no)
 			(do_not_autoplace no)
@@
 			)
 		)
-		(property "Footprint" "Resistor_SMD:R_Array_Convex_4x0603"
+		(property "Footprint" "Resistor_SMD:R_Array_Convex_4x1206"
 			(at 134.62 227.33 0)
 			(hide yes)

Commit message: WORKING ON POC - Proof of concept
Connections:
- net +3V3: now also U24.1, U25.1, U28.1, U29.1, U32.1, U33.1, U36.1, U37.1; no longer R100.1, R114.1, R116.1, R66.1, R68.1, R82.1, R84.1, R98.1
- net OT0: now also R66.1; no longer U24.2
- net OT1: now also R82.1; no longer U28.2
- net OT2: now also R98.1; no longer U32.2
- net OT3: now also R114.1; no longer U36.2
- net OT4: now also R68.1; no longer U25.2
- net OT5: now also R84.1; no longer U29.2
- net OT6: now also R100.1; no longer U33.2
- net OT7: now also R116.1; no longer U37.2
- net at R116.2: now also U37.2; no longer U37.1
- net at R66.2: now also U24.2; no longer U24.1
- net at R84.2: now also U29.2; no longer U29.1
- net at R100.2: now also U33.2; no longer U33.1
- net at R98.2: now also U32.2; no longer U32.1
- net at R82.2: now also U28.2; no longer U28.1
- net at R68.2: now also U25.2; no longer U25.1
- net at R114.2: now also U36.2; no longer U36.1

Commit message: WORKING ON POC - Proof of concept
Parts:
- added JP8: SolderJumper_2_Open, Jumper:SolderJumper-2_P1.3mm_Open_RoundedPad1.0x1.5mm, symbol Jumper:SolderJumper_2_Open
Connections:
- net +3V3: now also JP8.2 (B); no longer U38.16 (VDD)
- new net: JP8.1 (A), U38.16 (VDD)
Changed lines of the file:
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@@
 	(wire
 		(pts
-			(xy 179.07 143.51) (xy 179.07 148.59)
+			(xy 179.07 127) (xy 179.07 134.62)
 		)
 		(stroke
@@
 		)
 	)
+	(wire
+		(pts
+			(xy 179.07 144.78) (xy 179.07 148.59)
+		)
+		(stroke
+			(width 0)
+			(type default)
+		)
+	)
 	(label "outp7"
 		(at 314.96 124.46 90)
@@
 	)
 	(symbol
+		(lib_id "Jumper:SolderJumper_2_Open")
+		(at 179.07 139.7 90)
+		(unit 1)
+		(body_style 1)
+		(exclude_from_sim no)
+		(in_bom no)
+		(on_board yes)
+		(in_pos_files yes)
+		(dnp no)
+		(fields_autoplaced yes)
+		(property "Reference" "JP8"
+			(at 181.61 139.6999 90)
+			(show_name no)
+			(do_not_autoplace no)
+			(effects
+				(font
+					(size 1.27 1.27)
+				)
+				(justify right)
+			)
+		)
+		(property "Value" "SolderJumper_2_Open"
+			(at 175.26 139.7 0)
+			(hide yes)
+			(show_name no)
+			(do_not_autoplace no)
+			(effects
+				(font
+					(size 1.27 1.27)
+				)
+			)
+		)
+		(property "Footprint" "Jumper:SolderJumper-2_P1.3mm_Open_RoundedPad1.0x1.5mm"
+			(at 179.07 139.7 0)
+			(hide yes)
+			(show_name no)
+			(do_not_autoplace no)
+			(effects
+				(font
+					(size 1.27 1.27)
+				)
+			)
+		)
+		(property "Datasheet" ""
+			(at 186.69 139.7 0)
+			(hide yes)
+			(show_name no)
+			(do_not_autoplace no)
+			(effects
+				(font
+					(size 1.27 1.27)
+				)
+			)
+		)
+		(property "Description" "Solder Jumper, 2-pole, open"
+			(at 184.15 139.7 0)
+			(hide yes)
+			(show_name no)
+			(do_not_autoplace no)
+			(effects
+				(font
+					(size 1.27 1.27)
+				)
+			)
+		)
+		(pin "2"
+		)
+		(pin "1"
+		)
+		(instances
+			(project "TSC BW 16 V3 POC"
+				(path "/65a0f6c1-6a57-4cd2-a77c-79691e6171da/4b14fb8a-3fb3-4e56-ad25-b944ad295dd9"
+					(reference "JP8")
+					(unit 1)
+				)
+			)
+		)
+	)
+	(symbol
 		(lib_id "Device:R")
 		(at 76.2 73.66 180)
@@
 	(symbol
 		(lib_id "power:+3V3")
-		(at 179.07 143.51 0)
+		(at 179.07 127 0)
 		(unit 1)
 		(body_style 1)
@@
 		(dnp no)
 		(property "Reference" "#PWR0159"
-			(at 179.07 147.32 0)
+			(at 179.07 130.81 0)
 			(hide yes)
 			(show_name no)
@@
 		)
 		(property "Value" "+3V3"
-			(at 175.514 145.542 90)
+			(at 175.514 129.032 90)
 			(show_name no)
 			(do_not_autoplace no)
@@
 		)
 		(property "Footprint" ""
-			(at 179.07 143.51 0)
+			(at 179.07 127 0)
 			(hide yes)
 			(show_name no)
@@
 		)
 		(property "Datasheet" ""
-			(at 179.07 143.51 0)
+			(at 179.07 127 0)
 			(hide yes)
 			(show_name no)
@@
 		)
 		(property "Description" "Power symbol creates a global label with name \"+3V3\""
-			(at 179.07 143.51 0)
+			(at 179.07 127 0)
 			(hide yes)
 			(show_name no)

Commit message: WORKING ON POC - Proof of concept
Parts:
- D12, D16, D20, D8: footprint LED_SMD:LED_1206_3216Metric -> LED_SMD:LED_1206_3216Metric_Pad1.42x1.75mm_HandSolder
- R100, R104, R105, R108, R109, R114, R115, R116, R117, R120, R121, R60, R61, R66, R67, R68, R69, R72, R73, R76, R77, R82, R83, R84, R85, R88, R89, R92, R93, R98, R99: footprint Resistor_SMD:R_1206_3216Metric_Pad1.30x1.75mm_HandSolder -> Resistor_SMD:R_0603_1608Metric_Pad0.98x0.95mm_HandSolder
- R101: value 8.2k -> 470R; footprint Resistor_SMD:R_1206_3216Metric_Pad1.30x1.75mm_HandSolder -> Resistor_SMD:R_0603_1608Metric_Pad0.98x0.95mm_HandSolder
- RN1: footprint Resistor_SMD:R_Array_Convex_4x1206 -> Resistor_SMD:R_Array_Convex_4x0603
- RN2: footprint Resistor_SMD:R_Array_Convex_4x1206 -> Resistor_SMD:R_Array_Concave_4x0603
Changed lines of the file:
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@@
 	)
 	(junction
-		(at 302.26 130.81)
-		(diameter 0)
-		(color 0 0 0 0)
-	)
-	(junction
 		(at 137.16 237.49)
 		(diameter 0)
@@
 	)
 	(junction
+		(at 302.26 130.81)
+		(diameter 0)
+		(color 0 0 0 0)
+	)
+	(junction
 		(at 300.99 64.77)
 		(diameter 0)
@@
 			)
 		)
-		(property "Footprint" "Resistor_SMD:R_1206_3216Metric_Pad1.30x1.75mm_HandSolder"
+		(property "Footprint" "Resistor_SMD:R_0603_1608Metric_Pad0.98x0.95mm_HandSolder"
 			(at 73.66 135.128 90)
 			(hide yes)
@@
 			)
 		)
-		(property "Footprint" "Resistor_SMD:R_1206_3216Metric_Pad1.30x1.75mm_HandSolder"
+		(property "Footprint" "Resistor_SMD:R_0603_1608Metric_Pad0.98x0.95mm_HandSolder"
 			(at 74.93 166.878 90)
 			(hide yes)
@@
 			)
 		)
-		(property "Footprint" "Resistor_SMD:R_1206_3216Metric_Pad1.30x1.75mm_HandSolder"
+		(property "Footprint" "Resistor_SMD:R_0603_1608Metric_Pad0.98x0.95mm_HandSolder"
 			(at 324.612 157.48 90)
 			(hide yes)
@@
 			)
 		)
-		(property "Footprint" "Resistor_SMD:R_1206_3216Metric_Pad1.30x1.75mm_HandSolder"
+		(property "Footprint" "Resistor_SMD:R_0603_1608Metric_Pad0.98x0.95mm_HandSolder"
 			(at 98.552 93.98 90)
 			(hide yes)
@@
 			)
 		)
-		(property "Footprint" "Resistor_SMD:R_1206_3216Metric_Pad1.30x1.75mm_HandSolder"
+		(property "Footprint" "Resistor_SMD:R_0603_1608Metric_Pad0.98x0.95mm_HandSolder"
 			(at 72.39 69.088 90)
 			(hide yes)
@@
 			)
 		)
-		(property "Footprint" "Resistor_SMD:R_1206_3216Metric_Pad1.30x1.75mm_HandSolder"
+		(property "Footprint" "Resistor_SMD:R_0603_1608Metric_Pad0.98x0.95mm_HandSolder"
 			(at 302.768 71.12 90)
 			(hide yes)
@@
 			)
 		)
-		(property "Footprint" "LED_SMD:LED_1206_3216Metric"
+		(property "Footprint" "LED_SMD:LED_1206_3216Metric_Pad1.42x1.75mm_HandSolder"
 			(at 318.77 67.31 0)
 			(hide yes)
@@
 			)
 		)
-		(property "Footprint" "Resistor_SMD:R_1206_3216Metric_Pad1.30x1.75mm_HandSolder"
+		(property "Footprint" "Resistor_SMD:R_0603_1608Metric_Pad0.98x0.95mm_HandSolder"
 			(at 304.038 137.16 90)
 			(hide yes)
@@
 			)
 		)
-		(property "Footprint" "Resistor_SMD:R_1206_3216Metric_Pad1.30x1.75mm_HandSolder"
+		(property "Footprint" "Resistor_SMD:R_0603_1608Metric_Pad0.98x0.95mm_HandSolder"
 			(at 299.72 164.338 90)
 			(hide yes)
@@
 			)
 		)
-		(property "Footprint" "Resistor_SMD:R_1206_3216Metric_Pad1.30x1.75mm_HandSolder"
+		(property "Footprint" "Resistor_SMD:R_0603_1608Metric_Pad0.98x0.95mm_HandSolder"
 			(at 270.51 169.418 90)
 			(hide yes)
@@
 			)
 		)
-		(property "Footprint" "Resistor_SMD:R_1206_3216Metric_Pad1.30x1.75mm_HandSolder"
+		(property "Footprint" "Resistor_SMD:R_0603_1608Metric_Pad0.98x0.95mm_HandSolder"
 			(at 323.342 91.44 90)
 			(hide yes)
@@
 			)
 		)
-		(property "Footprint" "Resistor_SMD:R_1206_3216Metric_Pad1.30x1.75mm_HandSolder"
+		(property "Footprint" "Resistor_SMD:R_0603_1608Metric_Pad0.98x0.95mm_HandSolder"
 			(at 43.18 140.208 90)
 			(hide yes)
@@
 			)
 		)
-		(property "Footprint" "Resistor_SMD:R_1206_3216Metric_Pad1.30x1.75mm_HandSolder"
+		(property "Footprint" "Resistor_SMD:R_0603_1608Metric_Pad0.98x0.95mm_HandSolder"
 			(at 297.18 66.548 90)
 			(hide yes)
@@
 			)
 		)
-		(property "Footprint" "Resistor_SMD:R_1206_3216Metric_Pad1.30x1.75mm_HandSolder"
+		(property "Footprint" "Resistor_SMD:R_0603_1608Metric_Pad0.98x0.95mm_HandSolder"
 			(at 77.978 73.66 90)
 			(hide yes)
@@
 			)
 		)
-		(property "Footprint" "Resistor_SMD:R_1206_3216Metric_Pad1.30x1.75mm_HandSolder"
+		(property "Footprint" "Resistor_SMD:R_0603_1608Metric_Pad0.98x0.95mm_HandSolder"
 			(at 80.518 171.45 90)
 			(hide yes)
@@
 			)
 		)
-		(property "Footprint" "LED_SMD:LED_1206_3216Metric"
+		(property "Footprint" "LED_SMD:LED_1206_3216Metric_Pad1.42x1.75mm_HandSolder"
 			(at 320.04 133.35 0)
 			(hide yes)
@@
 			)
 		)
-		(property "Footprint" "Resistor_SMD:R_1206_3216Metric_Pad1.30x1.75mm_HandSolder"
+		(property "Footprint" "Resistor_SMD:R_0603_1608Metric_Pad0.98x0.95mm_HandSolder"
 			(at 98.552 128.27 90)
 			(hide yes)
@@
 			)
 		)
-		(property "Footprint" "LED_SMD:LED_1206_3216Metric"
+		(property "Footprint" "LED_SMD:LED_1206_3216Metric_Pad1.42x1.75mm_HandSolder"
 			(at 320.04 99.06 0)
 			(hide yes)
@@
 			)
 		)
-		(property "Footprint" "Resistor_SMD:R_1206_3216Metric_Pad1.30x1.75mm_HandSolder"
+		(property "Footprint" "Resistor_SMD:R_0603_1608Metric_Pad0.98x0.95mm_HandSolder"
 			(at 44.45 105.918 90)
 			(hide yes)
@@
 			)
 		)
-		(property "Footprint" "Resistor_SMD:R_1206_3216Metric_Pad1.30x1.75mm_HandSolder"
+		(property "Footprint" "Resistor_SMD:R_0603_1608Metric_Pad0.98x0.95mm_HandSolder"
 			(at 73.66 100.838 90)
 			(hide yes)
@@
 			)
 		)
-		(property "Footprint" "Resistor_SMD:R_1206_3216Metric_Pad1.30x1.75mm_HandSolder"
+		(property "Footprint" "Resistor_SMD:R_0603_1608Metric_Pad0.98x0.95mm_HandSolder"
 			(at 267.97 71.628 90)
 			(hide yes)
@@
 			)
 		)
-		(property "Footprint" "Resistor_SMD:R_1206_3216Metric_Pad1.30x1.75mm_HandSolder"
+		(property "Footprint" "Resistor_SMD:R_0603_1608Metric_Pad0.98x0.95mm_HandSolder"
 			(at 322.072 59.69 90)
 			(hide yes)
@@
 			)
 		)
-		(property "Footprint" "Resistor_SMD:R_1206_3216Metric_Pad1.30x1.75mm_HandSolder"
+		(property "Footprint" "Resistor_SMD:R_0603_1608Metric_Pad0.98x0.95mm_HandSolder"
 			(at 269.24 137.668 90)
 			(hide yes)
@@
 			)
 		)
-		(property "Footprint" "Resistor_SMD:R_1206_3216Metric_Pad1.30x1.75mm_HandSolder"
+		(property "Footprint" "Resistor_SMD:R_0603_1608Metric_Pad0.98x0.95mm_HandSolder"
 			(at 323.342 125.73 90)
 			(hide yes)
@@
 			)
 		)
-		(property "Footprint" "Resistor_SMD:R_1206_3216Metric_Pad1.30x1.75mm_HandSolder"
+		(property "Footprint" "Resistor_SMD:R_0603_1608Metric_Pad0.98x0.95mm_HandSolder"
 			(at 79.248 105.41 90)
 			(hide yes)
@@
 			)
 		)
-		(property "Footprint" "Resistor_SMD:R_Array_Convex_4x1206"
+		(property "Footprint" "Resistor_SMD:R_Array_Concave_4x0603"
 			(at 274.32 227.33 0)
 			(hide yes)
@@
 			)
 		)
-		(property "Footprint" "Resistor_SMD:R_1206_3216Metric_Pad1.30x1.75mm_HandSolder"
+		(property "Footprint" "Resistor_SMD:R_0603_1608Metric_Pad0.98x0.95mm_HandSolder"
 			(at 305.308 168.91 90)
 			(hide yes)
@@
 			)
 		)
-		(property "Footprint" "Resistor_SMD:R_1206_3216Metric_Pad1.30x1.75mm_HandSolder"
+		(property "Footprint" "Resistor_SMD:R_0603_1608Metric_Pad0.98x0.95mm_HandSolder"
 			(at 304.038 102.87 90)
 			(hide yes)
@@
 			)
 		)
-		(property "Footprint" "Resistor_SMD:R_1206_3216Metric_Pad1.30x1.75mm_HandSolder"
+		(property "Footprint" "Resistor_SMD:R_0603_1608Metric_Pad0.98x0.95mm_HandSolder"
 			(at 44.45 74.168 90)
 			(hide yes)
@@
 			)
 		)
-		(property "Footprint" "Resistor_SMD:R_1206_3216Metric_Pad1.30x1.75mm_HandSolder"
+		(property "Footprint" "Resistor_SMD:R_0603_1608Metric_Pad0.98x0.95mm_HandSolder"
 			(at 298.45 98.298 90)
 			(hide yes)
@@
 		(dnp no)
 		(property "Reference" "R101"
-			(at 298.196 128.778 90)
+			(at 298.196 128.27 90)
 			(show_name no)
 			(do_not_autoplace no)
@@
 			)
 		)
-		(property "Value" "8.2k"
-			(at 298.704 11.938 90)
+		(property "Value" "470R"
+			(at 298.45 130.81 90)
 			(show_name no)
 			(do_not_autoplace no)
@@
 			)
 		)
-		(property "Footprint" "Resistor_SMD:R_1206_3216Metric_Pad1.30x1.75mm_HandSolder"
+		(property "Footprint" "Resistor_SMD:R_0603_1608Metric_Pad0.98x0.95mm_HandSolder"
 			(at 298.45 132.588 90)
 			(hide yes)
@@
 			)
 		)
-		(property "Footprint" "LED_SMD:LED_1206_3216Metric"
+		(property "Footprint" "LED_SMD:LED_1206_3216Metric_Pad1.42x1.75mm_HandSolder"
 			(at 321.31 165.1 0)
 			(hide yes)
@@
 			)
 		)
-		(property "Footprint" "Resistor_SMD:R_1206_3216Metric_Pad1.30x1.75mm_HandSolder"
+		(property "Footprint" "Resistor_SMD:R_0603_1608Metric_Pad0.98x0.95mm_HandSolder"
 			(at 270.51 103.378 90)
 			(hide yes)
@@
 			)
 		)
-		(property "Footprint" "Resistor_SMD:R_1206_3216Metric_Pad1.30x1.75mm_HandSolder"
+		(property "Footprint" "Resistor_SMD:R_0603_1608Metric_Pad0.98x0.95mm_HandSolder"
 			(at 99.822 160.02 90)
 			(hide yes)
@@
 			)
 		)
-		(property "Footprint" "Resistor_SMD:R_1206_3216Metric_Pad1.30x1.75mm_HandSolder"
+		(property "Footprint" "Resistor_SMD:R_0603_1608Metric_Pad0.98x0.95mm_HandSolder"
 			(at 79.248 139.7 90)
 			(hide yes)
@@
 			)
 		)
-		(property "Footprint" "Resistor_SMD:R_Array_Convex_4x1206"
+		(property "Footprint" "Resistor_SMD:R_Array_Convex_4x0603"
 			(at 134.62 227.33 0)
 			(hide yes)
@@
 			)
 		)
-		(property "Footprint" "Resistor_SMD:R_1206_3216Metric_Pad1.30x1.75mm_HandSolder"
+		(property "Footprint" "Resistor_SMD:R_0603_1608Metric_Pad0.98x0.95mm_HandSolder"
 			(at 97.282 62.23 90)
 			(hide yes)
@@
 			)
 		)
-		(property "Footprint" "Resistor_SMD:R_1206_3216Metric_Pad1.30x1.75mm_HandSolder"
+		(property "Footprint" "Resistor_SMD:R_0603_1608Metric_Pad0.98x0.95mm_HandSolder"
 			(at 44.45 171.958 90)
 			(hide yes)

Commit message: WORKING ON POC - Proof of concept
Parts:
- R100, R101, R104, R105, R108, R109, R114, R115, R116, R117, R120, R121, R60, R61, R66, R67, R68, R69, R72, R73, R76, R77, R82, R83, R84, R85, R88, R89, R92, R93, R98, R99: footprint Resistor_SMD:R_0603_1608Metric_Pad0.98x0.95mm_HandSolder -> Resistor_SMD:R_1206_3216Metric_Pad1.30x1.75mm_HandSolder
- RN1: footprint Resistor_SMD:R_Array_Convex_4x0603 -> Resistor_SMD:R_Array_Convex_4x1206
- RN2: footprint Resistor_SMD:R_Array_Concave_4x0603 -> Resistor_SMD:R_Array_Convex_4x1206

Commit message: WORKING ON POC - Proof of concept
Parts:
- added D10, D13, D14, D17, D18, D21, D6, D9: B150-E3, Diode_SMD:D_SMA, symbol Diode:B150-E3
Connections:
- net PGND: now also D10.2 (A), D13.2 (A), D14.2 (A), D17.2 (A), D18.2 (A), D21.2 (A), D6.2 (A), D9.2 (A)
- net outp1: now also D14.1 (K)
- net outp2: now also D17.1 (K)
- net outp3: now also D18.1 (K)
- net outp4: now also D21.1 (K)
- net outp5: now also D6.1 (K)
- net outp6: now also D9.1 (K)
- net outp7: now also D10.1 (K)
- net outp8: now also D13.1 (K)
