File: TSC BW  Proof Of Concept V1/esp32_S3_mcu.kicad_sch (KiCad schematic)
At the start: 10 parts, among them J3 Free GPIO !pull-up, J4 Free GPIO pull-up, U3 ESP32-S3-WROOM-1

Commit message: WORKING ON POC - Proof of concept
Parts:
- added J19: 691312510002, Connector_Phoenix_MSTB:PhoenixContact_MSTBA_2,5_2-G-5,08_1x02_P5.08mm_Horizontal, symbol pluggable_terminal_connector_2:691312510002
Connections:
- net SCL: now also J19.1
- net SDA: now also J19.2
