File: TSC BW  Proof Of Concept V1/usb_c_to_uart.kicad_sch (KiCad schematic)
At the start: 20 parts, among them J14 USB_C_Receptacle_USB2.0_16P, Q20 SS8050, Q21 SS8050, SW1 SW_Push, SW2 SW_Push, U44 CH340C

Commit message: WORKING ON POC - Proof of concept
Parts:
- added JP6: SolderJumper_2_Open, Jumper:SolderJumper-2_P1.3mm_Open_RoundedPad1.0x1.5mm, symbol Jumper:SolderJumper_2_Open
Connections:
- net +5V: now also JP6.1 (A); no longer C23.1, D22.1 (K)
- new net: C23.1, D22.1 (K), JP6.2 (B)
Changed lines of the file:
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@@
 	(text "USB - TO - UART"
 		(exclude_from_sim no)
-		(at 67.564 37.592 0)
+		(at 71.374 22.098 0)
 		(effects
 			(font
@@
 	)
 	(junction
-		(at 77.47 55.88)
-		(diameter 0)
-		(color 0 0 0 0)
-	)
-	(junction
 		(at 44.45 93.98)
 		(diameter 0)
@@
 		(color 0 0 0 0)
 	)
+	(junction
+		(at 77.47 55.88)
+		(diameter 0)
+		(color 0 0 0 0)
+	)
 	(no_connect
 		(at 151.13 71.12)
@@
 	(wire
 		(pts
+			(xy 77.47 48.26) (xy 77.47 55.88)
+		)
+		(stroke
+			(width 0)
+			(type default)
+		)
+	)
+	(wire
+		(pts
 			(xy 53.34 120.65) (xy 54.61 120.65)
 		)
@@
 	(wire
 		(pts
-			(xy 77.47 54.61) (xy 77.47 55.88)
+			(xy 77.47 33.02) (xy 77.47 38.1)
 		)
 		(stroke
@@
 	)
 	(symbol
+		(lib_id "Jumper:SolderJumper_2_Open")
+		(at 77.47 43.18 270)
+		(unit 1)
+		(body_style 1)
+		(exclude_from_sim no)
+		(in_bom no)
+		(on_board yes)
+		(in_pos_files yes)
+		(dnp no)
+		(fields_autoplaced yes)
+		(property "Reference" "JP6"
+			(at 80.01 43.1799 90)
+			(show_name no)
+			(do_not_autoplace no)
+			(effects
+				(font
+					(size 1.27 1.27)
+				)
+				(justify left)
+			)
+		)
+		(property "Value" "SolderJumper_2_Open"
+			(at 81.28 43.18 0)
+			(hide yes)
+			(show_name no)
+			(do_not_autoplace no)
+			(effects
+				(font
+					(size 1.27 1.27)
+				)
+			)
+		)
+		(property "Footprint" "Jumper:SolderJumper-2_P1.3mm_Open_RoundedPad1.0x1.5mm"
+			(at 77.47 43.18 0)
+			(hide yes)
+			(show_name no)
+			(do_not_autoplace no)
+			(effects
+				(font
+					(size 1.27 1.27)
+				)
+			)
+		)
+		(property "Datasheet" ""
+			(at 69.85 43.18 0)
+			(hide yes)
+			(show_name no)
+			(do_not_autoplace no)
+			(effects
+				(font
+					(size 1.27 1.27)
+				)
+			)
+		)
+		(property "Description" "Solder Jumper, 2-pole, open"
+			(at 72.39 43.18 0)
+			(hide yes)
+			(show_name no)
+			(do_not_autoplace no)
+			(effects
+				(font
+					(size 1.27 1.27)
+				)
+			)
+		)
+		(pin "2"
+		)
+		(pin "1"
+		)
+		(instances
+			(project "TSC BW 16 V3 POC"
+				(path "/65a0f6c1-6a57-4cd2-a77c-79691e6171da/c74c7530-d8b4-4eb2-9788-6af0f5549dcd"
+					(reference "JP6")
+					(unit 1)
+				)
+			)
+		)
+	)
+	(symbol
 		(lib_id "Transistor_BJT:SS8050")
 		(at 219.71 62.23 0)
@@
 	(symbol
 		(lib_id "power:+5V")
-		(at 77.47 54.61 0)
+		(at 77.47 33.02 0)
 		(unit 1)
 		(body_style 1)
@@
 		(fields_autoplaced yes)
 		(property "Reference" "#PWR0215"
-			(at 77.47 58.42 0)
+			(at 77.47 36.83 0)
 			(hide yes)
 			(show_name no)
@@
 		)
 		(property "Value" "+5V"
-			(at 77.47 49.53 0)
+			(at 77.47 27.94 0)
 			(show_name no)
 			(do_not_autoplace no)
@@
 		)
 		(property "Footprint" ""
-			(at 77.47 54.61 0)
+			(at 77.47 33.02 0)
 			(hide yes)
 			(show_name no)
@@
 		)
 		(property "Datasheet" ""
-			(at 77.47 54.61 0)
+			(at 77.47 33.02 0)
 			(hide yes)
 			(show_name no)
@@
 		)
 		(property "Description" "Power symbol creates a global label with name \"+5V\""
-			(at 77.47 54.61 0)
-			(hide yes)
-			(show_name no)
+			(at 77.47 33.02 0)
+			(hide yes)
+			(show_name no)

Commit message: WORKING ON POC - Proof of concept
Other:
- moved on the sheet: C23
Changed lines of the file:
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@@
 	)
 	(junction
+		(at 77.47 55.88)
+		(diameter 0)
+		(color 0 0 0 0)
+	)
+	(junction
 		(at 64.77 58.42)
 		(diameter 0)
@@
 		(color 0 0 0 0)
 	)
-	(junction
-		(at 77.47 55.88)
-		(diameter 0)
-		(color 0 0 0 0)
-	)
 	(no_connect
 		(at 151.13 71.12)
@@
 	(wire
 		(pts
-			(xy 77.47 55.88) (xy 81.28 55.88)
+			(xy 77.47 55.88) (xy 83.82 55.88)
 		)
 		(stroke
@@
 	(symbol
 		(lib_id "power:GND")
-		(at 88.9 55.88 90)
+		(at 91.44 55.88 90)
 		(unit 1)
 		(body_style 1)
@@
 		(fields_autoplaced yes)
 		(property "Reference" "#PWR0216"
-			(at 95.25 55.88 0)
+			(at 97.79 55.88 0)
 			(hide yes)
 			(show_name no)
@@
 		)
 		(property "Value" "GND"
-			(at 92.71 55.8799 90)
+			(at 95.25 55.8799 90)
 			(show_name no)
 			(do_not_autoplace no)
@@
 		)
 		(property "Footprint" ""
-			(at 88.9 55.88 0)
+			(at 91.44 55.88 0)
 			(hide yes)
 			(show_name no)
@@
 		)
 		(property "Datasheet" ""
-			(at 88.9 55.88 0)
+			(at 91.44 55.88 0)
 			(hide yes)
 			(show_name no)
@@
 		)
 		(property "Description" "Power symbol creates a global label with name \"GND\" , ground"
-			(at 88.9 55.88 0)
+			(at 91.44 55.88 0)
 			(hide yes)
 			(show_name no)
@@
 	(symbol
 		(lib_id "Device:C")
-		(at 85.09 55.88 90)
+		(at 87.63 55.88 90)
 		(unit 1)
 		(body_style 1)
@@
 		(dnp no)
 		(property "Reference" "C23"
-			(at 81.28 54.102 0)
+			(at 83.82 54.102 0)
 			(show_name no)
 			(do_not_autoplace no)
@@
 		)
 		(property "Value" "100nF"
-			(at 88.138 54.864 0)
+			(at 90.678 54.864 0)
 			(show_name no)
 			(do_not_autoplace no)
@@
 		)
 		(property "Footprint" "Capacitor_SMD:C_1206_3216Metric"
-			(at 88.9 54.9148 0)
+			(at 91.44 54.9148 0)
 			(hide yes)
 			(show_name no)
@@
 		)
 		(property "Datasheet" ""
-			(at 85.09 55.88 0)
+			(at 87.63 55.88 0)
 			(hide yes)
 			(show_name no)
@@
 		)
 		(property "Description" "Unpolarized capacitor"
-			(at 85.09 55.88 0)
+			(at 87.63 55.88 0)
 			(hide yes)
 			(show_name no)

Commit message: WORKING ON POC - Proof of concept
Connections:
- net GND: now also J14.SH (SHIELD); no longer J14.S1 (SHIELD)
Changed lines of the file:
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@@
 		(pin "B12"
 		)
-		(pin "S1"
+		(pin "SH"
 		)
 		(pin "B1"
