File: TSC BW  Proof Of Concept V1/TSC BW 16 V3 POC.kicad_pcb (KiCad board)
At the start: 2 copper layers, 162 x 105 mm, 231 parts, among them J1 691312510002, J10 Micro_SD_Card_Det_Hirose_DM3AT, J13 Analog Inputs, J14 USB_C_Receptacle_USB2.0_16P, J17 691312510002, J18 RJ45_Hanrun_HR911105A_Horizon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, J2 CR1220_S8411_45R, J3 Free GPIO !pull-up, J4 Free GPIO pull-up, J5 Terminal Plug, J7 Terminal Plug, Q1 BC817, Q10 NCE60P10K, Q11 NCE60P10K, Q14 NCE60P10K, Q15 NCE60P10K, Q18 NCE60P10K, Q19 NCE60P10K, Q2 AO3401A, Q20 SS8050, Q21 SS8050, Q6 NCE60P10K, Q7 NCE60P10K, SW1 SW_Push, SW2 SW_Push, U1 XL1509-5.0, U10 PC357C, U11 PC357C, U14 PC357C, U15 PC357C, U18 PC357C, U19 PC357C, U2 AMS1117-3.3, U20 PCF8574T, U24 PC357C, U25 PC357C, U28 PC357C, U29 PC357C, U3 ESP32-S3-WROOM-1, U32 PC357C, U33 PC357C, U36 PC357C, U37 PC357C, U38 PCF8574T, U40 AT24CS04-SSHM, U41 DS3231MZ, U44 CH340C, U46 W5500, U48 MAX13487EESA, U6 PC357C, U7 PC357C, Y4 25M

Commit message: WORKING ON POC - Proof of concept
Parts:
- C47, C48, C49, C50, C51, C52, C53, C54, C55, C56, C57, C59, C61, C62, C63, C64, C65, C66: footprint Capacitor_SMD:C_1206_3216Metric -> Capacitor_SMD:C_0603_1608Metric_Pad1.08x0.95mm_HandSolder
- R183, R186, R188, R189, R190, R191, R192, R193, R194, R197, R198: footprint Resistor_SMD:R_1206_3216Metric_Pad1.30x1.75mm_HandSolder -> Resistor_SMD:R_0603_1608Metric_Pad0.98x0.95mm_HandSolder
- R184: footprint Resistor_SMD:R_1206_3216Metric_Pad1.30x1.75mm_HandSolder -> Resistor_SMD:R_0603_1608Metric
- RN10: footprint Resistor_SMD:R_Array_Convex_5x1206 -> Resistor_SMD:R_Array_Convex_5x0603
- RN3: footprint Resistor_SMD:R_Array_Convex_4x1206 -> Resistor_SMD:R_Array_Convex_4x0603
- moved C61 26.8 mm to (231.3, 134.3), turned to -90 degrees
- moved C64 25.5 mm to (211.6, 128.0), turned to -90 degrees
- moved RN3 24.1 mm to (211.8, 122.8)
- moved R194 23.9 mm to (229.2, 134.3), turned to 90 degrees
- moved C49 23.8 mm to (229.0, 110.0), turned to 90 degrees
- moved RN10 23.4 mm to (211.8, 118.3)
- moved C48 23.0 mm to (186.9, 122.7)
- moved C47 23.0 mm to (186.8, 112.9)
- moved R186 23.0 mm to (179.3, 117.5)
- moved Y4 23.0 mm to (187.3, 117.8)
- moved C63 21.3 mm to (214.7, 110.0), turned to 90 degrees
- moved C50 17.2 mm to (226.6, 110.0), turned to 90 degrees
- moved R190 17.0 mm to (218.3, 128.0), turned to -90 degrees
- moved R189 16.0 mm to (216.3, 128.0), turned to -90 degrees
- moved C62 15.7 mm to (217.1, 110.0), turned to 90 degrees
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
Commit message: WORKING ON POC - Proof of concept
Parts:
- moved C47 38.3 mm to (224.9, 110.1)
- moved Y4 33.4 mm to (220.0, 111.0), turned to 180 degrees
- moved C48 30.8 mm to (215.0, 110.0), turned to 0 degrees
- moved C63 3.94 mm to (213.7, 106.2)
- moved C62 3.90 mm to (216.3, 106.2)
- moved JP5 3.88 mm to (210.6, 106.2)
- moved C54 3.87 mm to (218.8, 106.2)
- moved C53 3.84 mm to (221.4, 106.2)
- moved C51 3.82 mm to (223.9, 106.2)
- moved C50 3.81 mm to (226.5, 106.2)
- moved C49 3.81 mm to (229.0, 106.2)
Changed lines of the file:
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@@
 	(footprint "Capacitor_SMD:C_0603_1608Metric_Pad1.08x0.95mm_HandSolder"
 		(layer "F.Cu")
-		(at 186.788 112.903 180)
+		(at 224.9435 110.109 180)
 		(descr "Capacitor SMD 0603 (1608 Metric), square (rectangular) end terminal, IPC-7351 nominal with elongated pad for handsoldering. (Body size source: IPC-SM-782 page 76, https://www.pcb-3d.com/wordpress/wp-content/uploads/ipc-sm-782a_amendment_1_and_2.pdf)")
 		(tags "capacitor handsolder")
@@
 			(at 0 1.43 180)
 			(layer "F.Fab")
+			(hide yes)
 			(effects
 				(font
@@
 	(footprint "Capacitor_SMD:C_0603_1608Metric_Pad1.08x0.95mm_HandSolder"
 		(layer "F.Cu")
-		(at 186.915 122.682 180)
+		(at 215.011 109.982)
 		(descr "Capacitor SMD 0603 (1608 Metric), square (rectangular) end terminal, IPC-7351 nominal with elongated pad for handsoldering. (Body size source: IPC-SM-782 page 76, https://www.pcb-3d.com/wordpress/wp-content/uploads/ipc-sm-782a_amendment_1_and_2.pdf)")
 		(tags "capacitor handsolder")
 		(property "Reference" "C48"
-			(at 0 -1.43 180)
+			(at 0 -1.43 0)
 			(layer "F.SilkS")
 			(effects
@@
 		)
 		(property "Value" "12pF"
-			(at 0 1.43 180)
+			(at 0 1.651 0)
 			(layer "F.Fab")
+			(hide yes)
 			(effects
 				(font
@@
 		)
 		(property "Datasheet" ""
-			(at 0 0 180)
+			(at 0 0 0)
 			(layer "F.Fab")
 			(hide yes)
@@
 		)
 		(property "Description" "Unpolarized capacitor"
-			(at 0 0 180)
+			(at 0 0 0)
 			(layer "F.Fab")
 			(hide yes)
@@
 		)
 		(property "KiLib_Generator" "SMD_2terminal_chip_molded"
-			(at 0 0 180)
+			(at 0 0 0)
 			(layer "F.SilkS")
 			(hide yes)
@@
 		(duplicate_pad_numbers_are_jumpers no)
 		(fp_line
-			(start -0.146267 0.51)
-			(end 0.146267 0.51)
+			(start -0.146267 -0.51)
+			(end 0.146267 -0.51)
 			(stroke
 				(width 0.12)
@@
 		)
 		(fp_line
-			(start -0.146267 -0.51)
-			(end 0.146267 -0.51)
+			(start -0.146267 0.51)
+			(end 0.146267 0.51)
 			(stroke
 				(width 0.12)
@@
 		)
 		(fp_text user "${REFERENCE}"
-			(at 0 0 180)
+			(at 0 0 0)
 			(layer "F.Fab")
 			(effects
@@
 		)
 		(pad "1" smd roundrect
-			(at -0.8625 0 180)
+			(at -0.8625 0)
 			(size 1.075 0.95)
 			(layers "F.Cu" "F.Mask" "F.Paste")
@@
 		)
 		(pad "2" smd roundrect
-			(at 0.8625 0 180)
+			(at 0.8625 0)
 			(size 1.075 0.95)
 			(layers "F.Cu" "F.Mask" "F.Paste")
@@
 	(footprint "Capacitor_SMD:C_0603_1608Metric_Pad1.08x0.95mm_HandSolder"
 		(layer "F.Cu")
-		(at 219.474143 110.0085 90)
+		(at 218.80453 106.1985 90)
 		(descr "Capacitor SMD 0603 (1608 Metric), square (rectangular) end terminal, IPC-7351 nominal with elongated pad for handsoldering. (Body size source: IPC-SM-782 page 76, https://www.pcb-3d.com/wordpress/wp-content/uploads/ipc-sm-782a_amendment_1_and_2.pdf)")
 		(tags "capacitor handsolder")
@@
 	(footprint "Capacitor_SMD:C_0603_1608Metric_Pad1.08x0.95mm_HandSolder"
 		(layer "F.Cu")
-		(at 217.097428 110.0085 90)
+		(at 216.255877 106.1985 90)
 		(descr "Capacitor SMD 0603 (1608 Metric), square (rectangular) end terminal, IPC-7351 nominal with elongated pad for handsoldering. (Body size source: IPC-SM-782 page 76, https://www.pcb-3d.com/wordpress/wp-content/uploads/ipc-sm-782a_amendment_1_and_2.pdf)")
 		(tags "capacitor handsolder")
@@
 	(footprint "Capacitor_SMD:C_0603_1608Metric_Pad1.08x0.95mm_HandSolder"
 		(layer "F.Cu")
-		(at 221.850857 110.0085 90)
+		(at 221.353184 106.1985 90)
 		(descr "Capacitor SMD 0603 (1608 Metric), square (rectangular) end terminal, IPC-7351 nominal with elongated pad for handsoldering. (Body size source: IPC-SM-782 page 76, https://www.pcb-3d.com/wordpress/wp-content/uploads/ipc-sm-782a_amendment_1_and_2.pdf)")
 		(tags "capacitor handsolder")
@@
 	(footprint "Capacitor_SMD:C_0603_1608Metric_Pad1.08x0.95mm_HandSolder"
 		(layer "F.Cu")
-		(at 214.720714 110.0085 90)
+		(at 213.707224 106.1985 90)
 		(descr "Capacitor SMD 0603 (1608 Metric), square (rectangular) end terminal, IPC-7351 nominal with elongated pad for handsoldering. (Body size source: IPC-SM-782 page 76, https://www.pcb-3d.com/wordpress/wp-content/uploads/ipc-sm-782a_amendment_1_and_2.pdf)")
 		(tags "capacitor handsolder")
@@
 	(footprint "Capacitor_SMD:C_0603_1608Metric_Pad1.08x0.95mm_HandSolder"
 		(layer "F.Cu")
-		(at 228.981 110.0085 90)
+		(at 228.999143 106.1985 90)
 		(descr "Capacitor SMD 0603 (1608 Metric), square (rectangular) end terminal, IPC-7351 nominal with elongated pad for handsoldering. (Body size source: IPC-SM-782 page 76, https://www.pcb-3d.com/wordpress/wp-content/uploads/ipc-sm-782a_amendment_1_and_2.pdf)")
 		(tags "capacitor handsolder")
@@
 	(footprint "Jumper:SolderJumper-2_P1.3mm_Open_RoundedPad1.0x1.5mm"
 		(layer "F.Cu")
-		(at 211.545714 109.967 -90)
+		(at 210.638571 106.1985 -90)
 		(descr "SMD Solder Jumper, 1x1.5mm, rounded Pads, 0.3mm gap, open")
 		(tags "solder jumper open")
@@
 	(footprint "Capacitor_SMD:C_0603_1608Metric_Pad1.08x0.95mm_HandSolder"
 		(layer "F.Cu")
-		(at 226.604285 110.0085 90)
+		(at 226.45049 106.1985 90)
 		(descr "Capacitor SMD 0603 (1608 Metric), square (rectangular) end terminal, IPC-7351 nominal with elongated pad for handsoldering. (Body size source: IPC-SM-782 page 76, https://www.pcb-3d.com/wordpress/wp-content/uploads/ipc-sm-782a_amendment_1_and_2.pdf)")
 		(tags "capacitor handsolder")
@@
 	(footprint "Capacitor_SMD:C_0603_1608Metric_Pad1.08x0.95mm_HandSolder"
 		(layer "F.Cu")
-		(at 224.227571 110.0085 90)
+		(at 223.901837 106.1985 90)
 		(descr "Capacitor SMD 0603 (1608 Metric), square (rectangular) end terminal, IPC-7351 nominal with elongated pad for handsoldering. (Body size source: IPC-SM-782 page 76, https://www.pcb-3d.com/wordpress/wp-content/uploads/ipc-sm-782a_amendment_1_and_2.pdf)")
 		(tags "capacitor handsolder")
@@
 		)
 		(embedded_fonts no)
-		(model "${KICAD10_3DMODEL_DIR}/Connector_RJ.3dshapes/RJ45_Hanrun_HR911105A_Horizontal.step"
+		(model "${KIPRJMOD}/3D models/HR911105A.step"
 			(offset
-				(xyz 0 0 0)
+				(xyz 4.5 -3.5 -0.5)
 			)
 			(scale
@@
 			)
 			(rotate
-				(xyz 0 0 0)
+				(xyz -90 -0 -180)
 			)
 		)
@@
 	(footprint "Crystal:Crystal_SMD_3225-4Pin_3.2x2.5mm"
 		(layer "F.Cu")
-		(at 187.286 117.772 -90)
+		(at 220.007 111.037 180)
 		(descr "SMD3225/4, Crystal, 3.2x2.5mm package, SMD, http://www.txccrystal.com/images/pdf/7m-accuracy.pdf")
 		(property "Reference" "Y4"
-			(at 0 -2.45 90)
+			(at 0 -2.45 0)
 			(layer "F.SilkS")
 			(effects
@@
 		)
 		(property "Value" "25M"
-			(at 0 2.45 90)
+			(at 0 2.45 0)
 			(layer "F.Fab")
+			(hide yes)
 			(effects
 				(font
@@
 		)
 		(property "Datasheet" ""
-			(at 0 0 90)
+			(at 0 0 0)
 			(layer "F.Fab")
 			(hide yes)
@@
 		)
 		(property "Description" "Two pin crystal"
-			(at 0 0 90)
+			(at 0 0 0)
 			(layer "F.Fab")
 			(hide yes)
@@
 		)
 		(property "KiLib_Generator" "crystal_resonator_oscillator"
-			(at 0 0 90)
+			(at 0 0 0)
 			(layer "F.SilkS")
 			(hide yes)
@@
 		)
 		(fp_text user "${REFERENCE}"
-			(at 0 0 90)
+			(at 0 0 0)
 			(layer "F.Fab")
 			(effects
@@
 		)
 		(pad "1" smd roundrect
-			(at -1.1 0.85 270)
+			(at -1.1 0.85 180)
 			(size 1.4 1.2)
 			(layers "F.Cu" "F.Mask" "F.Paste")
@@
 		)
 		(pad "2" smd roundrect
-			(at 1.1 0.85 270)
+			(at 1.1 0.85 180)
 			(size 1.4 1.2)
 			(layers "F.Cu" "F.Mask" "F.Paste")
@@
 		)
 		(pad "3" smd roundrect
-			(at 1.1 -0.85 270)
+			(at 1.1 -0.85 180)
 			(size 1.4 1.2)
 			(layers "F.Cu" "F.Mask" "F.Paste")
@@
 		)
 		(pad "4" smd roundrect
-			(at -1.1 -0.85 270)
+			(at -1.1 -0.85 180)
 			(size 1.4 1.2)
 			(layers "F.Cu" "F.Mask" "F.Paste")

Commit message: WORKING ON POC - Proof of concept
Parts:
- removed R42, R44, R46, R48, R50, R52, R54, R56: 4.7k, Resistor_SMD:R_1206_3216Metric_Pad1.30x1.75mm_HandSolder
- D12, D16, D20, D8: footprint LED_SMD:LED_1206_3216Metric -> LED_SMD:LED_1206_3216Metric_Pad1.42x1.75mm_HandSolder
- R100, R104, R105, R108, R109, R114, R115, R116, R117, R12, R120, R121, R13, R16, R17, R20, R21, R24, R25, R28, R29, R32, R33, R36, R37, R40, R41, R60, R61, R66, R67, R68, R69, R72, R73, R76, R77, R82, R83, R84, R85, R88, R89, R92, R93, R98, R99: footprint Resistor_SMD:R_1206_3216Metric_Pad1.30x1.75mm_HandSolder -> Resistor_SMD:R_0603_1608Metric_Pad0.98x0.95mm_HandSolder
- R101: value 8.2k -> 470R; footprint Resistor_SMD:R_1206_3216Metric_Pad1.30x1.75mm_HandSolder -> Resistor_SMD:R_0603_1608Metric_Pad0.98x0.95mm_HandSolder
- RN1: footprint Resistor_SMD:R_Array_Convex_4x1206 -> Resistor_SMD:R_Array_Convex_4x0603
- RN2: footprint Resistor_SMD:R_Array_Convex_4x1206 -> Resistor_SMD:R_Array_Concave_4x0603
- moved U37 388.0 mm to (232.0, 90.6), turned to 90 degrees
- moved U33 377.2 mm to (222.4, 90.6), turned to 90 degrees
- moved U29 366.3 mm to (212.4, 90.6), turned to 90 degrees
- moved R121 361.0 mm to (232.1, 82.8), turned to 180 degrees
- moved R117 360.5 mm to (232.1, 85.3), turned to 180 degrees
- moved R116 360.1 mm to (232.0, 95.6)
- moved R105 357.6 mm to (222.5, 82.8), turned to 180 degrees
- moved R101 357.0 mm to (222.5, 85.3), turned to 180 degrees
- moved R100 356.4 mm to (222.4, 95.6)
- moved U25 356.0 mm to (202.6, 90.4), turned to 90 degrees
- moved R89 353.7 mm to (212.4, 82.9), turned to 180 degrees
- moved R85 353.1 mm to (212.5, 85.3), turned to 180 degrees
- moved R84 352.4 mm to (212.4, 95.6)
- moved R73 350.3 mm to (202.7, 82.8), turned to 180 degrees
- moved R69 349.5 mm to (202.7, 85.3), turned to 180 degrees
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Connections:
- RN4 pad 5: /8 DIGITAL INPUTS/OT3 -> /8 DIGITAL INPUTS/IN_P3
- RN4 pad 6: /8 DIGITAL INPUTS/OT2 -> /8 DIGITAL INPUTS/IN_P2
- RN4 pad 7: /8 DIGITAL INPUTS/OT1 -> /8 DIGITAL INPUTS/IN_P1
- RN4 pad 8: /8 DIGITAL INPUTS/OT0 -> /8 DIGITAL INPUTS/IN_P0
- RN5 pad 5: /8 DIGITAL INPUTS/OT7 -> /8 DIGITAL INPUTS/IN_P7
- RN5 pad 6: /8 DIGITAL INPUTS/OT6 -> /8 DIGITAL INPUTS/IN_P6
- RN5 pad 7: /8 DIGITAL INPUTS/OT5 -> /8 DIGITAL INPUTS/IN_P5
- RN5 pad 8: /8 DIGITAL INPUTS/OT4 -> /8 DIGITAL INPUTS/IN_P4
Other:
- board size 162 x 105 mm -> 187.7 x 105 mm

Commit message: WORKING ON POC - Proof of concept
Parts:
- R100, R101, R104, R105, R108, R109, R114, R115, R116, R117, R12, R120, R121, R13, R16, R17, R20, R21, R24, R25, R28, R29, R32, R33, R36, R37, R40, R41, R60, R61, R66, R67, R68, R69, R72, R73, R76, R77, R82, R83, R84, R85, R88, R89, R92, R93, R98, R99: footprint Resistor_SMD:R_0603_1608Metric_Pad0.98x0.95mm_HandSolder -> Resistor_SMD:R_1206_3216Metric_Pad1.30x1.75mm_HandSolder
- RN1: footprint Resistor_SMD:R_Array_Convex_4x0603 -> Resistor_SMD:R_Array_Convex_4x1206
- RN2: footprint Resistor_SMD:R_Array_Concave_4x0603 -> Resistor_SMD:R_Array_Convex_4x1206
- moved U20 7.80 mm to (118.2, 94.4)
- moved RN4 7.80 mm to (128.9, 92.1)
- moved RN5 7.80 mm to (108.0, 92.1)
- moved R116 5.34 mm to (231.8, 101.0)
- moved R100 5.33 mm to (222.4, 101.0)
- moved R114 5.33 mm to (192.4, 101.0)
- moved R68 5.33 mm to (202.6, 101.0)
- moved R82 5.33 mm to (172.7, 101.0)
- moved R84 5.33 mm to (212.4, 101.0)
- moved R98 5.33 mm to (182.8, 101.0)
- moved R66 4.19 mm to (163.2, 101.0)
- moved U25 3.63 mm to (202.6, 94.1)
- moved U28 3.63 mm to (172.6, 94.1)
- moved U32 3.63 mm to (182.6, 94.1)
- moved U36 3.63 mm to (192.4, 94.1)
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
Commit message: WORKING ON POC - Proof of concept
Parts:
- added D10: B150-E3, Diode_SMD:D_SMA, F.Cu at (222.1, 65.0)
- added D13: B150-E3, Diode_SMD:D_SMA, F.Cu at (232.0, 65.0)
- added D14: B150-E3, Diode_SMD:D_SMA, F.Cu at (163.4, 65.2)
- added D17: B150-E3, Diode_SMD:D_SMA, F.Cu at (173.4, 65.2)
- added D18: B150-E3, Diode_SMD:D_SMA, F.Cu at (183.9, 65.0)
- added D21: B150-E3, Diode_SMD:D_SMA, F.Cu at (193.3, 65.2)
- added D6: B150-E3, Diode_SMD:D_SMA, F.Cu at (203.3, 65.0)
- added D9: B150-E3, Diode_SMD:D_SMA, F.Cu at (212.2, 65.0)
- added J19: 691312510002, Connector_Phoenix_MSTB:PhoenixContact_MSTBA_2,5_2-G-5,08_1x02_P5.08mm_Horizontal, F.Cu at (65.9, 144.1)
- moved R109 372.8 mm to (234.2, 59.0), turned to 90 degrees
- moved R93 369.6 mm to (224.4, 59.0), turned to 90 degrees
- moved D20 357.3 mm to (230.1, 59.0), turned to 90 degrees
- moved R77 355.8 mm to (214.1, 59.0), turned to 90 degrees
- moved R61 353.5 mm to (205.5, 59.0), turned to 90 degrees
- moved D16 346.4 mm to (220.2, 59.0), turned to 90 degrees
- moved JP8 335.9 mm to (201.7, 106.6)
- moved D12 335.5 mm to (210.2, 59.0), turned to 90 degrees
- moved R108 334.2 mm to (195.6, 59.0), turned to 90 degrees
- moved R92 331.3 mm to (186.2, 59.0), turned to 90 degrees
- moved R76 327.4 mm to (175.6, 59.0), turned to 90 degrees
- moved R5 326.1 mm to (171.2, 123.0), turned to -90 degrees
- moved D8 325.5 mm to (200.9, 59.0), turned to 90 degrees
- moved R6 321.5 mm to (167.3, 123.0), turned to -90 degrees
- moved D19 318.4 mm to (191.3, 59.2), turned to 90 degrees
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Other:
- board size 187.7 x 105 mm -> 177.4 x 113.6 mm

Commit message: WORKING ON POC - Proof of concept
Parts:
- moved U3 2.54 mm to (163.9, 143.2)
- moved J14 0.44 mm to (131.2, 150.2)
Connections:
- J10 pad SH: (no net) -> /SD CARD/CGND
- J14 pad SH: (no net) -> GND
Changed lines of the file:
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@@
 	)
 	(setup
+		(stackup
+			(layer "F.SilkS"
+				(type "Top Silk Screen")
+			)
+			(layer "F.Paste"
+				(type "Top Solder Paste")
+			)
+			(layer "F.Mask"
+				(type "Top Solder Mask")
+				(thickness 0.01)
+			)
+			(layer "F.Cu"
+				(type "copper")
+				(thickness 0.035)
+			)
+			(layer "dielectric 1"
+				(type "core")
+				(thickness 1.51)
+				(material "FR4")
+				(epsilon_r 4.5)
+				(loss_tangent 0.02)
+			)
+			(layer "B.Cu"
+				(type "copper")
+				(thickness 0.035)
+			)
+			(layer "B.Mask"
+				(type "Bottom Solder Mask")
+				(thickness 0.01)
+			)
+			(layer "B.Paste"
+				(type "Bottom Solder Paste")
+			)
+			(layer "B.SilkS"
+				(type "Bottom Silk Screen")
+			)
+			(copper_finish "None")
+			(dielectric_constraints no)
+		)
 		(pad_to_mask_clearance 0)
 		(allow_soldermask_bridges_in_footprints no)
@@
 	(footprint "Connector_USB:USB_C_Receptacle_GCT_USB4105-xx-A_16P_TopMnt_Horizontal"
 		(layer "F.Cu")
-		(at 131.189 149.801)
+		(at 131.191 150.241)
 		(descr "USB 2.0 Type C Receptacle, GCT, 16P, top mounted, horizontal, 5A: https://gct.co/files/drawings/usb4105.pdf")
 		(tags "USB C Type-C Receptacle SMD USB 2.0 16P 16C USB4105-15-A USB4105-15-A-060 USB4105-15-A-120 USB4105-GF-A USB4105-GF-A-060 USB4105-GF-A-120")
@@
 			(unit
 				(name "A")
-				(pins "S1" "A1" "A12" "B1" "B12" "A4" "A9" "B4" "B9" "A5" "B5" "A7" "B7"
+				(pins "SH" "A1" "A12" "B1" "B12" "A4" "A9" "B4" "B9" "A5" "B5" "A7" "B7"
 					"A6" "B6" "A8" "B8"
 				)
 			)
 		)
-		(attr smd)
 		(duplicate_pad_numbers_are_jumpers no)
 		(fp_line
@@
 			(layers "*.Cu" "*.Mask" "F.Paste")
 			(remove_unused_layers no)
+			(net "GND")
+			(pinfunction "SHIELD_SH")
+			(pintype "passive")
 		)
 		(pad "SH" thru_hole oval
@@
 			(layers "*.Cu" "*.Mask" "F.Paste")
 			(remove_unused_layers no)
+			(net "GND")
+			(pinfunction "SHIELD_SH")
+			(pintype "passive")
 		)
 		(pad "SH" thru_hole oval
@@
 			(layers "*.Cu" "*.Mask" "F.Paste")
 			(remove_unused_layers no)
+			(net "GND")
+			(pinfunction "SHIELD_SH")
+			(pintype "passive")
 		)
 		(pad "SH" thru_hole oval
@@
 			(layers "*.Cu" "*.Mask" "F.Paste")
 			(remove_unused_layers no)
+			(net "GND")
+			(pinfunction "SHIELD_SH")
+			(pintype "passive")
 		)
 		(embedded_fonts no)
@@
 	(footprint "RF_Module:ESP32-S3-WROOM-1"
 		(layer "F.Cu")
-		(at 165.59 141.321 180)
+		(at 163.857 143.179 180)
 		(descr "2.4 GHz Wi-Fi and Bluetooth module  https://www.espressif.com/sites/default/files/documentation/esp32-s3-wroom-1_wroom-1u_datasheet_en.pdf")
 		(tags "2.4 GHz Wi-Fi and Bluetooth module")
@@
 			(polygon
 				(pts
-					(xy 189.59 148.071) (xy 141.59 148.071) (xy 141.59 169.071) (xy 189.59 169.071)
+					(xy 187.857 149.929) (xy 139.857 149.929) (xy 139.857 170.929) (xy 187.857 170.929)
 				)
 			)
@@
 			(unit
 				(name "A")
-				(pins "1" "2" "3" "4" "5" "6" "7" "8" "10" "9" "11")
+				(pins "1" "2" "3" "4" "5" "6" "7" "8" "10" "9" "SH")
 			)
 		)
@@
 			(size 1 1.2)
 			(layers "F.Cu" "F.Mask" "F.Paste")
+			(net "/SD CARD/CGND")
+			(pinfunction "SH_SH")
+			(pintype "passive")
 		)
 		(pad "SH" smd rect
@@
 			(size 1 2.8)
 			(layers "F.Cu" "F.Mask" "F.Paste")
+			(net "/SD CARD/CGND")
+			(pinfunction "SH_SH")
+			(pintype "passive")
 		)
 		(pad "SH" smd rect
@@
 			(size 1 1.2)
 			(layers "F.Cu" "F.Mask" "F.Paste")
+			(net "/SD CARD/CGND")
+			(pinfunction "SH_SH")
+			(pintype "passive")
 		)
 		(pad "SH" smd rect
@@
 			(size 1.3 1.9)
 			(layers "F.Cu" "F.Mask" "F.Paste")
+			(net "/SD CARD/CGND")
+			(pinfunction "SH_SH")
+			(pintype "passive")
 		)
 		(zone

Commit message: WORKING ON POC - Proof of concept
Parts:
- moved C49 7.54 mm to (236.4, 104.7)
- moved C50 6.67 mm to (232.9, 104.6)
- moved C52 6.10 mm to (233.5, 111.0)
- moved C51 5.81 mm to (229.5, 104.5)
- moved C55 5.49 mm to (233.4, 114.7)
- moved R188 5.42 mm to (233.5, 122.0)
- moved C56 5.20 mm to (233.4, 118.3)
- moved C59 4.97 mm to (234.9, 127.5)
- moved C53 4.90 mm to (226.0, 104.6)
- moved R192 4.08 mm to (231.6, 127.5)
- moved C66 4.08 mm to (225.0, 127.5)
- moved C54 4.04 mm to (222.5, 104.6)
- moved C47 3.51 mm to (228.3, 111.0)
- moved R186 3.50 mm to (211.8, 107.5)
- moved C62 3.26 mm to (219.1, 104.5)
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Routing:
- net GND: track 0.00 -> 140.5 mm, vias 0 -> 4
- net +3V3 VW: track 0.00 -> 131.5 mm, vias 0 -> 4
- net /W500 v3/ActLed: track 0.00 -> 70.3 mm, vias 0 -> 2
- net /W500 v3/LinkedLed: track 0.00 -> 48.0 mm, vias 0 -> 2
- net /W500 v3/RCT: track 0.00 -> 33.0 mm
- net CGND: track 0.00 -> 24.4 mm
- net /W500 v3/TCT: track 0.00 -> 21.7 mm
- net Net-(RN10-R1.1): track 0.00 -> 21.1 mm, vias 0 -> 2
- net Net-(RN3-R4.2): track 0.00 -> 19.0 mm, vias 0 -> 2
- net /W500 v3/TD+: track 0.00 -> 17.8 mm
- net /W500 v3/TD-: track 0.00 -> 15.8 mm
- net Net-(RN3-R1.2): track 0.00 -> 14.4 mm, vias 0 -> 2
- net Net-(RN3-R2.2): track 0.00 -> 14.0 mm, vias 0 -> 2
- net Net-(RN3-R3.2): track 0.00 -> 13.9 mm, vias 0 -> 2
- net /W500 v3/RXP+: track 0.00 -> 13.8 mm
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
Commit message: WORKING ON POC - Proof of concept
Parts:
- moved JP7 13.9 mm to (82.8, 124.1)
- moved JP3 0.57 mm to (115.6, 119.2), turned to 90 degrees
- moved U38 0.19 mm to (191.1, 110.9)
Routing:
- net +3V3: track 0.00 -> 244.3 mm, vias 0 -> 2
- net GND: track 140.5 -> 264.5 mm, vias 4 -> 6
- net ETH_INT: track 0.00 -> 111.2 mm, vias 0 -> 6
- net ETH_RST: track 0.00 -> 101.1 mm, vias 0 -> 2
- net ETH_SCLK: track 0.00 -> 93.0 mm, vias 0 -> 4
- net ETH_SCS: track 0.00 -> 85.4 mm
- net ETH_MOSI: track 0.00 -> 66.4 mm, vias 0 -> 2
- net ETH_MISO: track 0.00 -> 65.7 mm, vias 0 -> 4
- net VinLoad1: track 0.00 -> 54.3 mm, vias 0 -> 2
- net /8 DIGITAL OUTPUTS/OT7: track 0.00 -> 53.1 mm
- net /8 DIGITAL OUTPUTS/OT6: track 0.00 -> 45.9 mm
- net /8 DIGITAL OUTPUTS/OT0: track 0.00 -> 39.7 mm
- net /8 DIGITAL OUTPUTS/OT5: track 0.00 -> 37.7 mm
- net /8 DIGITAL OUTPUTS/OT1: track 0.00 -> 33.4 mm
- net /8 DIGITAL OUTPUTS/OT4: track 0.00 -> 29.8 mm
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