File: TSC BW  Proof Of Concept V1/TSC BW 16 V3 POC.kicad_pcb (KiCad board)
At the start: 2 copper layers, 177.4 x 113.6 mm, 232 parts, among them J1 691312510002, J10 Micro_SD_Card_Det_Hirose_DM3AT, J13 Analog Inputs, J14 USB_C_Receptacle_USB2.0_16P, J17 691312510002, J18 RJ45_Hanrun_HR911105A_Horizon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, J19 691312510002, J2 CR1220_S8411_45R, J3 Free GPIO !pull-up, J4 Free GPIO pull-up, J5 Terminal Plug, J7 Terminal Plug, Q1 BC817, Q10 NCE60P10K, Q11 NCE60P10K, Q14 NCE60P10K, Q15 NCE60P10K, Q18 NCE60P10K, Q19 NCE60P10K, Q2 AO3401A, Q20 SS8050, Q21 SS8050, Q6 NCE60P10K, Q7 NCE60P10K, SW1 SW_Push, SW2 SW_Push, U1 XL1509-5.0, U10 PC357C, U11 PC357C, U14 PC357C, U15 PC357C, U18 PC357C, U19 PC357C, U2 AMS1117-3.3, U20 PCF8574T, U24 PC357C, U25 PC357C, U28 PC357C, U29 PC357C, U3 ESP32-S3-WROOM-1, U32 PC357C, U33 PC357C, U36 PC357C, U37 PC357C, U38 PCF8574T, U40 AT24CS04-SSHM, U41 DS3231MZ, U44 CH340C, U46 W5500, U48 MAX13487EESA, U6 PC357C, U7 PC357C, Y4 25M

Commit message: WORKING ON POC - Proof of concept
Routing:
- net /8 DIGITAL OUTPUTS/outp7: track 0.00 -> 38.2 mm
- net /8 DIGITAL OUTPUTS/outp8: track 0.00 -> 36.9 mm
- net /8 DIGITAL OUTPUTS/outp5: track 0.00 -> 29.1 mm
- net /8 DIGITAL OUTPUTS/outp6: track 0.00 -> 28.7 mm
- net PGND: track 0.00 -> 13.8 mm
- net Net-(D8-A): track 0.00 -> 4.58 mm
- net Net-(D16-A): track 0.00 -> 4.20 mm
- net Net-(D20-A): track 0.00 -> 4.07 mm
- net Net-(D12-A): track 0.00 -> 3.94 mm

Commit message: WORKING ON POC - Proof of concept
Parts:
- moved H2 84.5 mm to (107.8, 49.5)
- moved J5 7.37 mm to (158.0, 52.4)
- moved J19 5.48 mm to (71.4, 144.0)
- moved H4 4.29 mm to (66.9, 136.7)
- moved R197 1.51 mm to (229.5, 143.6)
- moved J10 1.33 mm to (198.3, 145.9)
- moved J1 1.02 mm to (70.0, 52.2)
- moved J3 0.74 mm to (70.9, 116.9)
- moved J13 0.71 mm to (98.9, 52.3)
- moved J4 0.52 mm to (70.9, 97.4)
- moved H3 0.52 mm to (232.6, 150.6)
- moved J14 0.44 mm to (131.3, 150.7)
- moved J7 0.22 mm to (215.8, 52.2)
- moved U3 0.12 mm to (163.5, 141.8)
Routing:
- net GND: track 264.5 -> 0.00 mm, vias 6 -> 0
- net +3V3: track 244.3 -> 0.00 mm, vias 2 -> 0
- net +3V3 VW: track 136.5 -> 0.00 mm, vias 4 -> 0
- net ETH_INT: track 111.2 -> 0.00 mm, vias 6 -> 0
- net ETH_RST: track 101.1 -> 0.00 mm, vias 2 -> 0
- net ETH_SCLK: track 93.0 -> 0.00 mm, vias 4 -> 0
- net ETH_SCS: track 85.4 -> 0.00 mm
- net /W500 v3/ActLed: track 70.3 -> 0.00 mm, vias 2 -> 0
- net ETH_MOSI: track 66.4 -> 0.00 mm, vias 2 -> 0
- net ETH_MISO: track 65.7 -> 0.00 mm, vias 4 -> 0
- net VinLoad1: track 54.3 -> 0.00 mm, vias 2 -> 0
- net /8 DIGITAL OUTPUTS/OT7: track 53.1 -> 0.00 mm
- net /W500 v3/LinkedLed: track 48.0 -> 0.00 mm, vias 2 -> 0
- net /8 DIGITAL OUTPUTS/OT6: track 45.9 -> 0.00 mm
- net /8 DIGITAL OUTPUTS/OT0: track 39.7 -> 0.00 mm
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
Commit message: WORKING ON POC - Proof of concept
Parts:
- moved JP4 22.1 mm to (188.7, 111.9)
- moved R153 22.1 mm to (117.8, 120.1)
- moved D25 22.1 mm to (125.6, 120.8)
- moved C27 22.1 mm to (85.3, 46.2)
- moved C28 22.1 mm to (79.1, 46.2)
- moved C43 22.1 mm to (140.6, 95.0)
- moved C47 22.1 mm to (219.2, 90.8)
- moved C48 22.1 mm to (207.3, 90.5)
- moved C50 22.1 mm to (223.8, 84.5)
- moved C52 22.1 mm to (224.4, 90.8)
- moved C53 22.1 mm to (216.9, 84.5)
- moved C59 22.1 mm to (225.8, 107.3)
- moved C64 22.1 mm to (199.4, 107.5)
- moved C66 22.1 mm to (215.9, 107.3)
- moved D12 22.1 mm to (201.1, 38.8)
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Routing:
- net GND: track 0.00 -> 872.0 mm, vias 0 -> 8
- net +3V3: track 0.00 -> 519.2 mm, vias 0 -> 7
- net PGND: track 0.00 -> 281.7 mm, vias 0 -> 2
- net SCL: track 0.00 -> 222.4 mm, vias 0 -> 5
- net SDA: track 0.00 -> 188.5 mm, vias 0 -> 6
- net ANALOG_A3: track 0.00 -> 148.5 mm, vias 0 -> 2
- net ANALOG_A4: track 0.00 -> 139.6 mm, vias 0 -> 2
- net ANALOG_A2: track 0.00 -> 138.4 mm, vias 0 -> 2
- net +3V3 VW: track 0.00 -> 135.9 mm, vias 0 -> 4
- net ANALOG_A1: track 0.00 -> 128.7 mm, vias 0 -> 2
- net +5V: track 0.00 -> 115.3 mm, vias 0 -> 4
- net /ESP32 S3 MCU/F_IO47: track 0.00 -> 113.5 mm, vias 0 -> 2
- net VinLoad1: track 0.00 -> 113.2 mm
- net /8 DIGITAL INPUTS/PGND: track 0.00 -> 107.7 mm
- net 485RX: track 0.00 -> 104.7 mm, vias 0 -> 2
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- added copper zone on B.Cu, net GND

Commit message: WORKING ON POC - Proof of concept
Routing:
- net +3V3 VW: track 135.9 -> 145.4 mm, vias 4 -> 6
- net /W500 v3/RD+: track 10.6 -> 11.7 mm
- net /W500 v3/TD+: track 18.1 -> 18.7 mm
- net /W500 v3/TD-: track 14.7 -> 15.2 mm
Changed lines of the file:
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@@
 	(segment
 		(start 202.7302 106.355)
-		(end 205.9849 106.355)
+		(end 204.56 106.355)
 		(width 0.25)
 		(layer "F.Cu")
@@
 	)
 	(segment
+		(start 204.56 106.355)
+		(end 204.56 108.37)
+		(width 0.25)
+		(layer "F.Cu")
+		(net "+3V3 VW")
+	)
+	(segment
 		(start 201.5505 90.3925)
 		(end 201.5505 93.3175)
@@
 	)
 	(segment
+		(start 209.45 106.1946)
+		(end 209.2896 106.355)
+		(width 0.25)
+		(layer "F.Cu")
+		(net "+3V3 VW")
+	)
+	(segment
 		(start 202.1665 85.3175)
 		(end 206.4755 85.3175)
@@
 	)
 	(segment
+		(start 204.56 108.37)
+		(end 204.58 108.39)
+		(width 0.25)
+		(layer "F.Cu")
+		(net "+3V3 VW")
+	)
+	(segment
+		(start 204.56 106.355)
+		(end 205.9849 106.355)
+		(width 0.25)
+		(layer "F.Cu")
+		(net "+3V3 VW")
+	)
+	(segment
+		(start 209.45 105.21)
+		(end 209.45 106.1946)
+		(width 0.25)
+		(layer "F.Cu")
+		(net "+3V3 VW")
+	)
+	(segment
 		(start 216.726 99.6675)
 		(end 217.838 99.6675)
@@
 	)
 	(via
+		(at 209.45 105.21)
+		(size 0.6)
+		(drill 0.3)
+		(layers "F.Cu" "B.Cu")
+		(net "+3V3 VW")
+	)
+	(via
 		(at 213.1939 101.7534)
 		(size 0.6)
@@
 	)
 	(via
+		(at 204.58 108.39)
+		(size 0.6)
+		(drill 0.3)
+		(layers "F.Cu" "B.Cu")
+		(net "+3V3 VW")
+	)
+	(via
 		(at 220.5072 91.8522)
 		(size 0.6)
@@
 	)
 	(segment
+		(start 204.58 108.39)
+		(end 206.27 108.39)
+		(width 0.25)
+		(layer "B.Cu")
+		(net "+3V3 VW")
+	)
+	(segment
 		(start 215.6167 99.3306)
 		(end 215.6167 99.2562)
@@
 	)
 	(segment
+		(start 206.27 108.39)
+		(end 209.45 105.21)
+		(width 0.25)
+		(layer "B.Cu")
+		(net "+3V3 VW")
+	)
+	(segment
 		(start 217.3345 97.5384)
 		(end 217.3345 95.0249)
@@
 	)
 	(segment
-		(start 208.5146 106.0754)
-		(end 208.51362 106.07638)
-		(width 0.2)
-		(layer "F.Cu")
-		(net "/W500 v3/TD+")
-	)
-	(segment
-		(start 207.89 106.840586)
-		(end 207.89 107.06)
-		(width 0.2)
-		(layer "F.Cu")
-		(net "/W500 v3/TD+")
-	)
-	(segment
-		(start 208.51362 106.216966)
-		(end 207.89 106.840586)
+		(start 211.3755 103.13)
+		(end 211.3755 103.89991)
 		(width 0.2)
 		(layer "F.Cu")
@@
 	)
 	(segment
-		(start 207.89 107.06)
-		(end 209.01 108.18)
-		(width 0.2)
-		(layer "F.Cu")
-		(net "/W500 v3/TD+")
-	)
-	(segment
-		(start 208.5146 105.875778)
-		(end 208.5146 106.0754)
-		(width 0.2)
-		(layer "F.Cu")
-		(net "/W500 v3/TD+")
-	)
-	(segment
-		(start 208.822878 105.5675)
-		(end 208.5146 105.875778)
+		(start 211.4255 103.08)
+		(end 211.3755 103.13)
 		(width 0.2)
 		(layer "F.Cu")
@@
 	)
 	(segment
-		(start 211.4255 103.08)
-		(end 211.3755 103.13)
-		(width 0.2)
-		(layer "F.Cu")
-		(net "/W500 v3/TD+")
-	)
-	(segment
-		(start 209.818993 104.57)
-		(end 208.822878 105.566115)
+		(start 210.70541 104.57)
+		(end 208.875686 104.57)
 		(width 0.2)
 		(layer "F.Cu")
@@
 	)
 	(segment
-		(start 205.8704 116.8175)
-		(end 207.96 114.7279)
+		(start 207.89 105.555686)
+		(end 207.89 107.06)
 		(width 0.2)
 		(layer "F.Cu")
@@
 	)
 	(segment
-		(start 210.70541 104.57)
-		(end 209.818993 104.57)
+		(start 208.875686 104.57)
+		(end 207.89 105.555686)
 		(width 0.2)
 		(layer "F.Cu")
@@
 	)
 	(segment
-		(start 208.51362 106.07638)
-		(end 208.51362 106.216966)
+		(start 205.8704 116.8175)
+		(end 207.96 114.7279)
 		(width 0.2)
 		(layer "F.Cu")
@@
 	)
 	(segment
-		(start 211.3755 103.13)
-		(end 211.3755 103.89991)
-		(width 0.2)
-		(layer "F.Cu")
-		(net "/W500 v3/TD+")
-	)
-	(segment
-		(start 208.822878 105.566115)
-		(end 208.822878 105.5675)
+		(start 207.89 107.06)
+		(end 209.01 108.18)
 		(width 0.2)
 		(layer "F.Cu")
@@
 	)
 	(segment
-		(start 208.11362 106.05128)
-		(end 205.9849 108.18)
+		(start 210.9255 103.08)
+		(end 210.97452 103.12902)
 		(width 0.2)
 		(layer "F.Cu")
@@
 	)
 	(segment
-		(start 208.11362 105.709687)
-		(end 208.11362 106.05128)
+		(start 210.97452 103.12902)
+		(end 210.97452 103.69548)
 		(width 0.2)
 		(layer "F.Cu")
@@
 	)
 	(segment
-		(start 207.54 109.7351)
-		(end 205.9849 108.18)
+		(start 208.71 104.17)
+		(end 207.44 105.44)
 		(width 0.2)
 		(layer "F.Cu")
@@
 	)
 	(segment
-		(start 210.5 104.17)
-		(end 209.653307 104.17)
+		(start 207.54 109.7351)
+		(end 205.9849 108.18)
 		(width 0.2)
 		(layer "F.Cu")
@@
 	)
 	(segment
-		(start 207.54 113.635)
-		(end 207.54 109.7351)
+		(start 210.5 104.17)
+		(end 208.71 104.17)
 		(width 0.2)
 		(layer "F.Cu")
@@
 	)
 	(segment
-		(start 206.8975 114.2775)
-		(end 207.54 113.635)
+		(start 207.44 105.44)
+		(end 207.44 106.7249)
 		(width 0.2)
 		(layer "F.Cu")
@@
 	)
 	(segment
-		(start 209.653307 104.17)
-		(end 208.11362 105.709687)
+		(start 207.54 113.635)
+		(end 207.54 109.7351)
 		(width 0.2)
 		(layer "F.Cu")
@@
 	)
 	(segment
-		(start 210.97452 103.12902)
-		(end 210.97452 103.69548)
+		(start 206.8975 114.2775)
+		(end 207.54 113.635)
 		(width 0.2)
 		(layer "F.Cu")
@@
 	)
 	(segment
-		(start 210.9255 103.08)
-		(end 210.97452 103.12902)
+		(start 207.44 106.7249)
+		(end 205.9849 108.18)
 		(width 0.2)
 		(layer "F.Cu")
@@
 	)
 	(segment
-		(start 208.1775 116.8175)
-		(end 208.4028 116.8175)
+		(start 208.4028 116.8175)
+		(end 210.7075 114.5128)
+		(width 0.2)
+		(layer "F.Cu")
+		(net "/W500 v3/RD+")
+	)
+	(segment
+		(start 210.7075 113.6825)
+		(end 213.93 110.46)
 		(width 0.2)
 		(layer "F.Cu")
@@
 	(segment
 		(start 210.7075 114.5128)
-		(end 210.7075 110.0668)
+		(end 210.7075 113.6825)
+		(width 0.2)
+		(layer "F.Cu")
+		(net "/W500 v3/RD+")
+	)
+	(segment
+		(start 208.1775 116.8175)
+		(end 208.4028 116.8175)
 		(width 0.2)
 		(layer "F.Cu")
@@
 	)
 	(segment
-		(start 210.7075 110.0668)
+		(start 213.93 109.5157)
 		(end 212.5943 108.18)
 		(width 0.2)
@@
 	)
 	(segment
-		(start 208.4028 116.8175)
-		(end 210.7075 114.5128)
+		(start 213.93 110.46)
+		(end 213.93 109.5157)
 		(width 0.2)
 		(layer "F.Cu")
@@
 	)
 	(segment
-		(start 215.8989 108.18)
-		(end 215.8989 110.3561)
+		(start 214.33 109.63)
+		(end 214.33 110.625686)
+		(width 0.2)
+		(layer "F.Cu")
+		(net "/W500 v3/RD-")
+	)
+	(segment
+		(start 215.78 108.18)
+		(end 214.33 109.63)
 		(width 0.2)
 		(layer "F.Cu")
@@
 	)
 	(segment
-		(start 215.8989 110.3561)
+		(start 214.33 110.625686)
+		(end 211.9775 112.978186)
+		(width 0.2)
+		(layer "F.Cu")
+		(net "/W500 v3/RD-")
+	)
+	(segment
+		(start 211.9775 112.978186)
 		(end 211.9775 114.2775)
 		(width 0.2)
 		(layer "F.Cu")
+		(net "/W500 v3/RD-")
+	)
+	(segment
+		(start 215.8989 108.18)
+		(end 215.78 108.18)
+		(width 0.2)
+		(layer "F.Cu")
