File: TSC BW  Proof Of Concept V1/not used schematics/Ethernet_W5500.kicad_sch (KiCad schematic)
At the start: 36 parts, among them J18 RJ45_Hanrun_HR911105A_Horizon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, U46 W5500, Y4 25M

Commit message: Proof Of Concept
Parts:
- removed C47, C48: 12pF, Capacitor_SMD:C_1206_3216Metric, symbol Device:C
- removed C49, C50, C51, C52, C53, C54, C64: 100nF, Capacitor_SMD:C_1206_3216Metric, symbol Device:C
- removed C55, C59: 10nF, Capacitor_SMD:C_1206_3216Metric, symbol Device:C
- removed C56: 4.7uF/6.3V, Capacitor_SMD:C_1206_3216Metric, symbol Device:C
- removed C57: 22nF, Capacitor_SMD:C_1206_3216Metric, symbol Device:C
- removed C61: 102/1KV, Capacitor_SMD:C_1206_3216Metric, symbol Device:C
- removed C62, C63: 10uF/10v, Capacitor_SMD:C_1206_3216Metric, symbol Device:C
- removed C65, C66: 6.8nF, Capacitor_SMD:C_1206_3216Metric, symbol Device:C
- removed J18: RJ45_Hanrun_HR911105A_Horizontal, external_lib:RJ45_Hanrun_HR911105A_Horizontal_3D, symbol Connector:RJ45_Hanrun_HR911105A_Horizontal
- removed R183, R184, R186: 10K, Resistor_SMD:R_1206_3216Metric_Pad1.30x1.75mm_HandSolder, symbol Device:R
- removed R185: 0R, Resistor_SMD:R_1206_3216Metric_Pad1.30x1.75mm_HandSolder, symbol Device:R
- removed R188: 12.4k 1%, Resistor_SMD:R_1206_3216Metric_Pad1.30x1.75mm_HandSolder, symbol Device:R
- removed R189, R190: 49R9, Resistor_SMD:R_1206_3216Metric_Pad1.30x1.75mm_HandSolder, symbol Device:R
- removed R191: 10R, Resistor_SMD:R_1206_3216Metric_Pad1.30x1.75mm_HandSolder, symbol Device:R
- removed R192, R193: 82R, Resistor_SMD:R_1206_3216Metric_Pad1.30x1.75mm_HandSolder, symbol Device:R
- removed R194: 1M, Resistor_SMD:R_1206_3216Metric_Pad1.30x1.75mm_HandSolder, symbol Device:R
- removed R197, R198: 1k, Resistor_SMD:R_1206_3216Metric_Pad1.30x1.75mm_HandSolder, symbol Device:R
- removed RN10: 10K R_Pack05, Resistor_SMD:R_Array_Convex_5x1206, symbol Device:R_Pack05
- removed RN3: R_Pack04, Resistor_SMD:R_Array_Convex_4x1206, symbol Device:R_Pack04
- removed U46: W5500, Package_QFP:LQFP-48_7x7mm_P0.5mm, symbol Interface_Ethernet:W5500
- removed Y4: 25M, Crystal:Crystal_SMD_3225-4Pin_3.2x2.5mm, symbol Device:Crystal
- added C28, C29: 20pF, Capacitor_SMD:C_1206_3216Metric, symbol Device:C
- added C30, C31, C32, C33, C34, C41: 100nF, Capacitor_SMD:C_1206_3216Metric, symbol Device:C
- added C35: 102/1KV, Capacitor_SMD:C_1206_3216Metric, symbol Device:C
- added C36: 4.7uF/6.3V, Capacitor_SMD:C_1206_3216Metric, symbol Device:C
- added C37: 22nF, Capacitor_SMD:C_1206_3216Metric, symbol Device:C
- added C38, C39: 6.8nF, Capacitor_SMD:C_1206_3216Metric, symbol Device:C
- added C40, C42: 10nF, Capacitor_SMD:C_1206_3216Metric, symbol Device:C
- added J16: RJ45_Hanrun_HR911105A_Horizontal, external_lib:RJ45_Hanrun_HR911105A_Horizontal_3D, symbol Connector:RJ45_Hanrun_HR911105A_Horizontal
- added R164, R165: 330R, Resistor_SMD:R_1206_3216Metric_Pad1.30x1.75mm_HandSolder, symbol Device:R
- added R169: 12.4k 1%, Resistor_SMD:R_1206_3216Metric_Pad1.30x1.75mm_HandSolder, symbol Device:R
- added R170: 0R, Resistor_SMD:R_1206_3216Metric_Pad1.30x1.75mm_HandSolder, symbol Device:R
- added R171, R175, R176, R182: 10K, Resistor_SMD:R_1206_3216Metric_Pad1.30x1.75mm_HandSolder, symbol Device:R
- added R172: 1M, Resistor_SMD:R_1206_3216Metric_Pad1.30x1.75mm_HandSolder, symbol Device:R
- added R173, R174: 510R, Resistor_SMD:R_1206_3216Metric_Pad1.30x1.75mm_HandSolder, symbol Device:R
- added R177, R178: 49R9, Resistor_SMD:R_1206_3216Metric_Pad1.30x1.75mm_HandSolder, symbol Device:R
- added R179: 10R, Resistor_SMD:R_1206_3216Metric_Pad1.30x1.75mm_HandSolder, symbol Device:R
- added R180, R181: 82R, Resistor_SMD:R_1206_3216Metric_Pad1.30x1.75mm_HandSolder, symbol Device:R
- added RN7: 10K R_Pack05, symbol Device:R_Pack05
- added RN8: 10K R_Pack03, symbol Device:R_Pack03
- added U45: W5500, Package_QFP:LQFP-48_7x7mm_P0.5mm, symbol Interface_Ethernet:W5500
- added Y3: 25M, symbol Device:Crystal
Connections:
- net +3V3: now also R170.2
- net +3V3 VW: now also C30.1, C31.1, C32.1, C33.1, C34.1, C41.2, R164.2, R165.2, R170.1, R171.2, R175.1, R176.1, R177.1, R178.1, R179.2, RN8.4 (R3.2), RN8.5 (R2.2), RN8.6 (R1.2), U45.11 (AVDD), U45.15 (AVDD), U45.17 (AVDD), U45.21 (AVDD), U45.28 (VDD), U45.4 (AVDD), U45.8 (AVDD)
- net ActLed: now also R173.1, U45.27 (ACTLED)
- net CGND: now also C35.2, J16.SH, R172.1
- net ETH_INT: now also R176.2, U45.36 (~{INT})
- net ETH_MISO: now also U45.34 (MISO)
- net ETH_MOSI: now also U45.35 (MOSI)
- net ETH_RST: now also R175.2, U45.37 (~{RST})
- net ETH_SCLK: now also U45.33 (SCLK)
- net ETH_SCS: now also R171.1, U45.32 (~{SCS})
- net GND: now also C28.1, C29.1, C30.2, C31.2, C32.2, C33.2, C34.2, C35.1, C36.2, C37.2, C40.1, C41.1, C42.1, J16.8, R169.2, R172.2, R182.2, RN7.10 (R1.2), RN7.6 (R5.2), RN7.7 (R4.2), RN7.8 (R3.2), RN7.9 (R2.2), U45.14 (AGND), U45.16 (AGND), U45.19 (AGND), U45.29 (GND), U45.3 (AGND), U45.48 (AGND), U45.9 (AGND)
- net LinkedLed: now also R174.1, U45.25 (LINKLED)
- net RCT: now also C40.2, J16.5 (RCT), R180.1, R181.2
- net RD+: now also C38.2, J16.3 (RD+), R180.2
- net RD-: now also C39.2, J16.6 (RD-), R181.1
- net RXN-: now also C39.1, U45.5 (RXN)
- net RXP+: now also C38.1, U45.6 (RXP)
- net TCT: now also C37.1, J16.4 (TCT), R179.1
- net TD+: now also J16.1 (TD+), R178.2, U45.2 (TXP)
- net TD-: now also J16.2 (TD-), R177.2, U45.1 (TXN)
- net X0: now also C29.2, U45.31 (XO), Y3.2
- net X1: now also C28.2, U45.30 (XI/CLKIN), Y3.1
- new net: J16.10, R173.2
- new net: J16.11, R174.2
- new net: J16.12, R164.1
- new net: J16.9, R165.1
- new net: RN7.1 (R1.1), U45.42 (RSVD)
- new net: RN7.2 (R2.1), U45.41 (RSVD)
- new net: RN7.3 (R3.1), U45.40 (RSVD)
- new net: RN7.4 (R4.1), U45.39 (RSVD)
- new net: RN7.5 (R5.1), U45.38 (RSVD)
- new net: RN8.1 (R1.1), U45.43 (PMODE2)
- new net: RN8.2 (R2.1), U45.44 (PMODE1)
- new net: RN8.3 (R3.1), U45.45 (PMODE0)
- new net: R169.1, U45.10 (EXRES1)
- new net: C36.1, U45.20 (TOCAP)
- new net: C42.2, U45.22 (1V2O)
- new net: R182.1, U45.23 (RSVD)
Other:
- note added: "ETHERNET GLOBAL PINS / LABELS P15"
- note added: "Ethernet (W5500) ETH_SCLK - PIN35 : GPIO42 ETH_MOSI - PIN37 : GPIO43 ETH_MISO - PIN36 : GPIO44 ETH_SCS - PIN8 : GPIO15 ETH_INT - PIN38 : GPIO2 ETH_RST - PIN39 : GPIO1"
- note removed: "GLOBAL PINS / LABELS"
- note removed: "ethernet: type: W5500 clk_pin: GPIO42 mosi_pin: GPIO43 miso_pin: GPIO44 cs_pin: GPIO15 interrupt_pin: GPIO2 reset_pin: GPIO1"
- company: (none) -> Tivana Holdings
- title: (none) -> TSC BW 16 V3.1
